File: ProofOfConcepts/AntennaPOC/schematic/schematic.sch (KiCad schematic (older format))
At the start: 0 parts

Commit message: schematic done
Connections:
- wire segments 48 -> 55
Changed lines of the file:
@@
 $Descr USLetter 11000 8500
 encoding utf-8
-Sheet 1 6
+Sheet 1 3
 Title ""
 Date ""
@@
 F6 "DRIVER_N" I L 7350 2500 50
 F7 "DRIVER_P" I L 7350 2400 50
-F8 "VCC_UNREGULATED" I L 7350 1950 50
-F9 "TEMP_SENSE_1" I L 7350 2700 50
-F10 "TEMP_SENSE_2" I L 7350 2800 50
-F11 "TEMP_SENSE_3" I L 7350 2900 50
+F8 "TEMP_SENSE_1_P" I L 7350 2700 50
+F9 "TEMP_SENSE_2_N" I L 7350 3000 50
+F10 "TEMP_SENSE_3_N" I L 7350 3200 50
+F11 "TEMP_SENSE_1_N" I L 7350 2800 50
+F12 "TEMP_SENSE_2_P" I L 7350 2900 50
+F13 "TEMP_SENSE_3_P" I L 7350 3100 50
 $EndSheet
 $Sheet
@@
 F10 "PELTIER_N" I R 3300 2650 50
 $EndSheet
-$Sheet
-S 4300 1400 1800 1100
-U 61F4C378
-F0 "Power Management" 50
-F1 "pwrmngmt.sch" 50
-F2 "BATT_IN" I L 4300 1700 50
-F3 "GND" I L 4300 2450 50
-F4 "3V3" I R 6100 1800 50
-F5 "VCC_UNREGULATED" I R 6100 2100 50
-F6 "PWR_SW_P" I L 4300 1900 50
-F7 "PWR_SW_N" I L 4300 2000 50
-F8 "VUSB" I L 4300 1450 50
-$EndSheet
 Wire Wire Line
 	4300 1450 3300 1450
@@
 Wire Wire Line
 	6700 2150 7350 2150
-$Sheet
-S 3900 3100 2450 1450
-U 6200D680
-F0 "Peltier Driver" 50
-F1 "driver.sch" 50
-F2 "DRIVER_P" I R 6350 3550 50
-F3 "DRIVER_N" I R 6350 3650 50
-F4 "PELTIER_P" I L 3900 3550 50
-F5 "PELTIER_N" I L 3900 3700 50
-F6 "VCC_UNREGULATED" I R 6350 3300 50
-F7 "GND" I L 3900 4500 50
-$EndSheet
+Wire Wire Line
+	7350 4800 7300 4800
+Wire Wire Line
+	7300 4800 7300 3200
+Wire Wire Line
+	7300 3200 7350 3200
+Wire Wire Line
+	7350 3100 7250 3100
+Wire Wire Line
+	7250 3100 7250 4900
+Wire Wire Line
+	7250 4900 7350 4900
+Wire Wire Line
+	7350 5050 7200 5050
+Wire Wire Line
+	7200 5050 7200 3000
+Wire Wire Line
+	7200 3000 7350 3000
 Wire Wire Line
 	7350 2900 7150 2900
@@
 L power:+3V3 #PWR0142
 U 1 1 622D92B4
-P 9300 5200
-F 0 "#PWR0142" H 9300 5050 50  0001 C CNN
-F 1 "+3V3" H 9315 5373 50  0000 C CNN
-F 2 "" H 9300 5200 50  0001 C CNN
-F 3 "" H 9300 5200 50  0001 C CNN
-	1    9300 5200
+P 9300 4800
+F 0 "#PWR0142" H 9300 4650 50  0001 C CNN
+F 1 "+3V3" H 9315 4973 50  0000 C CNN
+F 2 "" H 9300 4800 50  0001 C CNN
+F 3 "" H 9300 4800 50  0001 C CNN
+	1    9300 4800
 	1    0    0    -1
 $EndComp
@@
 L power:GND #PWR0143
 U 1 1 622DA41E
-P 9300 5300
-F 0 "#PWR0143" H 9300 5050 50  0001 C CNN
-F 1 "GND" H 9305 5127 50  0000 C CNN
-F 2 "" H 9300 5300 50  0001 C CNN
-F 3 "" H 9300 5300 50  0001 C CNN
-	1    9300 5300
+P 9300 4900
+F 0 "#PWR0143" H 9300 4650 50  0001 C CNN
+F 1 "GND" H 9305 4727 50  0000 C CNN
+F 2 "" H 9300 4900 50  0001 C CNN
+F 3 "" H 9300 4900 50  0001 C CNN
+	1    9300 4900
 	-1   0    0    -1
 $EndComp
 Wire Wire Line
-	9200 5300 9300 5300
-Wire Wire Line
-	9300 5200 9200 5200
-Wire Wire Line
-	7350 1950 6600 1950
-Wire Wire Line
-	6600 1950 6600 2100
-Connection ~ 6600 2100
-$Sheet
-S 7350 4400 1850 1400
-U 622394A9
-F0 "Temperature Sensors" 50
-F1 "tempsensor.sch" 50
-F2 "TEMP_SENSE_1" I L 7350 5400 50
-F3 "TEMP_SENSE_2" I L 7350 5300 50
-F4 "TEMP_SENSE_3" I L 7350 5150 50
-F5 "TEMP_SENSE_PWR" I R 9200 5200 50
-F6 "GND" I R 9200 5300 50
-$EndSheet
+	9200 4900 9300 4900
+Wire Wire Line
+	9300 4800 9200 4800
 $EndSCHEMATC
