File: ProofOfConcepts/AntennaPOC/schematic/MCU.kicad_sch (KiCad schematic)
At the start: 19 parts, among them J1 Conn_01x14_Male, J2 Conn_01x10_Male, J3 Conn_01x10_Male, J5 Conn_01x14_Male, U1 ESP32-D-WD-V3, Y1 Crystal_GND24

Commit message: s
Connections:
- net +3V3: now also U1.19 (VDD3P3_RTC); no longer U1.17 (GPIO14/MTMS)
- net at J2.10 (Pin_10): now also U1.24 (GPIO4); no longer U1.22 (GPIO2)
- net at J2.2 (Pin_2): now also U1.15 (GPIO26)
- net at J2.3 (Pin_3): now also U1.16 (GPIO27)
- net at J2.4 (Pin_4): now also U1.17 (GPIO14/MTMS); no longer U1.15 (GPIO26)
- net at J2.5 (Pin_5): now also U1.18 (GPIO12/MTDI); no longer U1.16 (GPIO27)
- net at J2.6 (Pin_6): now also U1.20 (GPIO13/MTCK); no longer U1.18 (GPIO12/MTDI)
- net at J2.7 (Pin_7): now also U1.21 (GPIO15/MTDO); no longer U1.19 (VDD3P3_RTC)
- net at J2.8 (Pin_8): now also U1.22 (GPIO2); no longer U1.20 (GPIO13/MTCK)
- net at J2.9 (Pin_9): now also U1.23 (GPIO0); no longer U1.21 (GPIO15/MTDO)
Other:
- moved on the sheet: C8, J2
