File: ProofOfConcepts/AntennaPOC/schematic/schematic.kicad_pcb (KiCad board)
At the start: 2 copper layers, 94 x 52.1 mm, 19 parts, among them J1 Conn_01x14_Male, J2 Conn_01x10_Male, J3 Conn_01x10_Male, J5 Conn_01x14_Male, U1 ESP32-D-WD-V3, Y1 Crystal_GND24

Commit message: 4
Other:
- net class Default removed

Commit message: s
Connections:
- AE1 pad 2: Net-(AE1-Pad2) -> unconnected-(AE1-Pad2)
- J1 pad 11: Net-(J1-Pad11) -> unconnected-(J1-Pad11)
- J1 pad 12: Net-(J1-Pad12) -> unconnected-(J1-Pad12)
- J1 pad 13: Net-(J1-Pad13) -> unconnected-(J1-Pad13)
- J1 pad 14: Net-(J1-Pad14) -> unconnected-(J1-Pad14)
- J2 pad 1: Net-(J2-Pad1) -> unconnected-(J2-Pad1)
- J5 pad 1: Net-(J5-Pad1) -> unconnected-(J5-Pad1)
