File: schematic/schematic.kicad_pcb (KiCad board)
At the start: 2 copper layers, 67.3 x 52.1 mm, 88 parts, among them J2 USB_C_Receptacle_USB2.0, J3 Peltier Connection, J4 Serial, SW1 Power Switch, U1 ESP32-D-WD-V3, U10 BSD316, U11 BSD316, U12 PC817, U13 PC817, U14 PC817, U15 AS431, U16 LM324, U17 XL6009, U18 PAM2305CGFADJ, U2 PC817, U3 BUK9K52-60E, U4 BUK9K52-60E, U6 PC817, U7 PC817, U8 PC817, U9 BSD316, Y1 Crystal_GND24

Commit message: e
Parts:
- removed R35, R36: 1k, Resistor_SMD:R_0805_2012Metric_Pad1.20x1.40mm_HandSolder
- removed R37, R38: 12.5k, Resistor_SMD:R_0805_2012Metric_Pad1.20x1.40mm_HandSolder
- added R4: .1, Resistor_SMD:R_1206_3216Metric_Pad1.30x1.75mm_HandSolder, F.Cu at (116.9, 92.9)
- added R5: 1k, Resistor_SMD:R_0805_2012Metric_Pad1.20x1.40mm_HandSolder, F.Cu at (122.3, 92.7)
- added R6: 1k, Resistor_SMD:R_0805_2012Metric_Pad1.20x1.40mm_HandSolder, F.Cu at (116.3, 96.0)
- added R7: 12.5k, Resistor_SMD:R_0805_2012Metric_Pad1.20x1.40mm_HandSolder, F.Cu at (116.3, 99.0)
- added U5: LM324, Package_SO:SOIC-14_3.9x8.7mm_P1.27mm, F.Cu at (109.7, 96.3)
- D4: footprint Diode_SMD:D_SMC_Handsoldering -> Diode_SMD:D_SMA_Handsoldering
- L3: footprint Inductor_SMD:L_12x12mm_H4.5mm -> Inductor_SMD:L_10.4x10.4_H4.8
- R34: value .1 -> 12.5k; footprint Resistor_SMD:R_1206_3216Metric_Pad1.30x1.75mm_HandSolder -> Resistor_SMD:R_0805_2012Metric_Pad1.20x1.40mm_HandSolder
- U12, U13, U14, U2, U6, U7, U8: footprint Package_SO:SOP-4_3.8x4.1mm_P2.54mm -> 1KicadLib:SMT_4_8.2x2.54
- U15: footprint Package_TO_SOT_SMD:SOT-23-5_HandSoldering -> Package_TO_SOT_SMD:SOT-23
- moved C6 13.5 mm to (152.2, 126.6)
- moved C7 13.5 mm to (148.4, 126.6)
- moved R34 13.5 mm to (137.2, 96.9)
- moved R39 13.5 mm to (144.3, 125.4)
- moved R9 13.5 mm to (129.8, 89.4)
- moved U16 13.5 mm to (135.9, 102.9)
- moved AE1 13.5 mm to (168.0, 118.3)
- moved C1 13.5 mm to (165.7, 121.7)
- moved C11 13.5 mm to (149.6, 93.1)
- moved C15 13.5 mm to (144.5, 110.4)
- moved C16 13.5 mm to (145.1, 115.9)
- moved C18 13.5 mm to (146.7, 118.9)
- moved C2 13.5 mm to (164.3, 123.1)
- moved C21 13.5 mm to (141.4, 110.4)
- moved C3 13.5 mm to (153.3, 127.3)
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Connections:
- BT3 pad 2: GND -> Net-(BT3-Pad2)
- R34 pad 2: GND -> Net-(U17-Pad5)
- U11 pad 4: GND -> Net-(BT3-Pad2)
- U16 pad 1: Net-(R38-Pad2) -> (no net)
- U16 pad 2: Net-(R35-Pad1) -> (no net)
- U16 pad 3: Net-(R36-Pad1) -> (no net)
- U17 pad 1: Net-(R34-Pad1) -> GND
- U17 pad 5: Net-(R38-Pad2) -> Net-(U17-Pad5)
Routing:
- net VCC_UNREGULATED: track 101.2 -> 214.1 mm, vias 2 -> 10
- net DRIVER_P: track 57.6 -> 0.00 mm, vias 2 -> 0
- net Vdrive: track 40.9 -> 0.00 mm
- net Net-(R34-Pad1): track 21.5 -> 0.00 mm, vias 1 -> 0
- net +BATT: track 29.5 -> 51.0 mm, vias 4 -> 5
- net CELL_MEAS_3: track 24.7 -> 43.7 mm, vias 2 -> 4
- net CELL_MEAS_2: track 19.0 -> 0.00 mm, vias 2 -> 0
- net /Peltier Driver/PELTIER_N: track 7.61 -> 0.00 mm, vias 2 -> 0
- net Net-(BT1-Pad2): track 16.0 -> 23.2 mm, vias 1 -> 2
- net (no net): track 0.00 -> 6.82 mm, vias 0 -> 2
- net /Peltier Driver/PELTIER_P: track 6.37 -> 0.00 mm, vias 2 -> 0
- net Net-(R38-Pad2): track 5.42 -> 0.00 mm, vias 1 -> 0
- net Net-(U17-Pad5): track 0.00 -> 5.42 mm, vias 0 -> 1
- net Net-(R35-Pad1): track 5.12 -> 0.00 mm, vias 1 -> 0
- net Net-(U12-Pad3): track 4.84 -> 0.00 mm
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Other:
- board size 67.3 x 52.1 mm -> 99.1 x 99.1 mm

Commit message: d
Parts:
- removed AE1: Antenna_Chip, RF_Antenna:Johanson_2450AT18x100
- removed BT1, BT2, BT3: Battery_Cell, Connector_PinHeader_2.54mm:PinHeader_1x02_P2.54mm_Vertical
- removed C1: 3.797pF, Capacitor_SMD:C_0805_2012Metric_Pad1.18x1.45mm_HandSolder
- removed C10, C21, C5, C8: 100nF, Capacitor_SMD:C_0805_2012Metric_Pad1.18x1.45mm_HandSolder
- removed C11, C15, C17, C9: 10uF, Capacitor_SMD:C_0805_2012Metric_Pad1.18x1.45mm_HandSolder
- removed C16: 100uF, Capacitor_SMD:C_1210_3225Metric_Pad1.33x2.70mm_HandSolder
- removed C18: 1uF, Capacitor_SMD:C_0805_2012Metric_Pad1.18x1.45mm_HandSolder
- removed C2: 4.64pF, Capacitor_SMD:C_0805_2012Metric_Pad1.18x1.45mm_HandSolder
- removed C20: Cfw (DNP), Capacitor_SMD:C_0805_2012Metric_Pad1.18x1.45mm_HandSolder
- removed C3: 3.3nF, Capacitor_SMD:C_0805_2012Metric_Pad1.18x1.45mm_HandSolder
- removed C4: 10nF, Capacitor_SMD:C_0805_2012Metric_Pad1.18x1.45mm_HandSolder
- removed C6, C7: 10pF, Capacitor_SMD:C_0805_2012Metric_Pad1.18x1.45mm_HandSolder
- removed D1, D2: LL4148, Diode_SMD:D_MiniMELF
- removed D4: SS34, Diode_SMD:D_SMA_Handsoldering
- removed J2: USB_C_Receptacle_USB2.0, 1KicadLib:USB4125-GF-A
- removed J3: Peltier Connection, Connector_PinHeader_2.54mm:PinHeader_1x02_P2.54mm_Vertical
- removed J4: Serial, Connector_PinHeader_2.54mm:PinHeader_1x03_P2.54mm_Vertical
- removed L1: 1.807nH, Inductor_SMD:L_0805_2012Metric_Pad1.15x1.40mm_HandSolder
- removed L2: 10uH NR8040T100M, Inductor_SMD:L_Taiyo-Yuden_NR-80xx_HandSoldering
- removed L3: 33uH, Inductor_SMD:L_10.4x10.4_H4.8
- removed R1: 20k, Resistor_SMD:R_0805_2012Metric_Pad1.20x1.40mm_HandSolder
- removed R10, R11, R2, R3: 300, Resistor_SMD:R_0805_2012Metric_Pad1.20x1.40mm_HandSolder
- removed R12, R15, R16: 28.7, Resistor_SMD:R_2512_6332Metric_Pad1.40x3.35mm_HandSolder
- removed R13: 33k, Resistor_SMD:R_0805_2012Metric_Pad1.20x1.40mm_HandSolder
- removed R14: 7.5k, Resistor_SMD:R_0805_2012Metric_Pad1.20x1.40mm_HandSolder
- removed R17, R18, R19: 200, Resistor_SMD:R_0805_2012Metric_Pad1.20x1.40mm_HandSolder
- removed R20, R21, R24: 90k, Resistor_SMD:R_0805_2012Metric_Pad1.20x1.40mm_HandSolder
- removed R22, R40: 100k, Resistor_SMD:R_0805_2012Metric_Pad1.20x1.40mm_HandSolder
- removed R23: 22k, Resistor_SMD:R_0805_2012Metric_Pad1.20x1.40mm_HandSolder
- removed R25: 390, Resistor_SMD:R_0805_2012Metric_Pad1.20x1.40mm_HandSolder
- removed R26: 180k, Resistor_SMD:R_0805_2012Metric_Pad1.20x1.40mm_HandSolder
- removed R27, R29: 68k, Resistor_SMD:R_0805_2012Metric_Pad1.20x1.40mm_HandSolder
- removed R28, R31: 56k, Resistor_SMD:R_0805_2012Metric_Pad1.20x1.40mm_HandSolder
- removed R30: 220k, Resistor_SMD:R_0805_2012Metric_Pad1.20x1.40mm_HandSolder
- removed R32: 120, Resistor_SMD:R_0805_2012Metric_Pad1.20x1.40mm_HandSolder
- removed R33: 500, Resistor_SMD:R_0805_2012Metric_Pad1.20x1.40mm_HandSolder
- removed R34, R7: 12.5k, Resistor_SMD:R_0805_2012Metric_Pad1.20x1.40mm_HandSolder
- removed R39: 150k, Resistor_SMD:R_0805_2012Metric_Pad1.20x1.40mm_HandSolder
- removed R4: .1, Resistor_SMD:R_1206_3216Metric_Pad1.30x1.75mm_HandSolder
- removed R5, R6: 1k, Resistor_SMD:R_0805_2012Metric_Pad1.20x1.40mm_HandSolder
- removed R8, R9: 5.1k, Capacitor_SMD:C_0805_2012Metric_Pad1.18x1.45mm_HandSolder
- removed SW1: Power Switch, Connector_PinHeader_2.54mm:PinHeader_1x02_P2.54mm_Vertical
- removed TH1, TH2, TH3: SDNT2012X103F3950FTF, Resistor_SMD:R_0805_2012Metric_Pad1.20x1.40mm_HandSolder
- removed U1: ESP32-D-WD-V3, Package_DFN_QFN:QFN-48-1EP_5x5mm_P0.35mm_EP3.7x3.7mm
- removed U10, U11, U9: BSD316, Package_TO_SOT_SMD:SOT-363_SC-70-6_Handsoldering
- removed U12, U13, U14, U2, U6, U7, U8: PC817, 1KicadLib:SMT_4_8.2x2.54
- removed U15: AS431, Package_TO_SOT_SMD:SOT-23
- removed U16, U5: LM324, Package_SO:SOIC-14_3.9x8.7mm_P1.27mm
- removed U17: XL6009, Package_TO_SOT_SMD:TO-263-5_TabPin3
- removed U18: PAM2305CGFADJ, Package_DFN_QFN:DFN-6-1EP_2x2mm_P0.65mm_EP1x1.6mm
- removed U3, U4: BUK9K52-60E, 1KicadLib:LFPAK56D
- removed Y1: Crystal_GND24, Crystal:Crystal_SMD_SeikoEpson_FA238-4Pin_3.2x2.5mm_HandSoldering
Routing:
- net VCC_UNREGULATED: track 214.1 -> 0.00 mm, vias 10 -> 0
- net +3V3: track 117.4 -> 0.00 mm, vias 10 -> 0
- net DRIVER_N: track 61.0 -> 0.00 mm, vias 2 -> 0
- net VBUS: track 54.7 -> 0.00 mm, vias 10 -> 0
- net TEMP_SENSE_1: track 52.7 -> 0.00 mm, vias 2 -> 0
- net +BATT: track 51.0 -> 0.00 mm, vias 5 -> 0
- net PWM: track 44.9 -> 0.00 mm, vias 2 -> 0
- net CELL_MEAS_3: track 43.7 -> 0.00 mm, vias 4 -> 0
- net TEMP_SENSE_2: track 36.3 -> 0.00 mm, vias 2 -> 0
- net Net-(BT1-Pad2): track 23.2 -> 0.00 mm, vias 2 -> 0
- net TEMP_SENSE_3: track 22.9 -> 0.00 mm, vias 2 -> 0
- net CELL_MEAS_1: track 20.6 -> 0.00 mm, vias 2 -> 0
- net Net-(D4-Pad2): track 18.6 -> 0.00 mm, vias 3 -> 0
- net Net-(BT2-Pad2): track 15.8 -> 0.00 mm, vias 1 -> 0
- net TXD: track 13.2 -> 0.00 mm
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- removed copper zone on B.Cu, net GND
- removed copper zone on F.Cu, net GND
Other:
- outline, holes or cut-outs redrawn
- board text removed: "GUANTANAMO BAY"
- board text removed: "Joesphan Lu"
