File: schematic/schematic.kicad_pcb (KiCad board)
At the start: 2 copper layers, 99.1 x 99.1 mm, 87 parts, among them J1 Peltier Connection, J2 USB_C_Receptacle_USB2.0, J3 Conn_01x01_Male, J4 Serial, J5 Conn_01x01_Male, J6 Conn_01x01_Male, J7 Conn_01x01_Male, J8 Conn_01x01_Male, SW1 Power Switch, U1 ESP32-D-WD-V3, U10 BSD316, U11 BSD316, U12 PC817, U13 PC817, U14 PC817, U15 AS431, U16 AP63203WU, U17 XL6009, U18 slg55021, U19 HT75xx-1-SOT89, U2 NL17SZ14, U3 DMT3020LSDQ, U4 DMT3020LSDQ, U5 LM324, U6 slg55021, U7 NL17SZ14, U8 NL17SZ14, U9 BSD316, Y1 Crystal_GND24

Commit message: e
Parts:
- added C16: 100nF, Capacitor_SMD:C_0805_2012Metric_Pad1.18x1.45mm_HandSolder, F.Cu at (132.3, 96.9)
- added C17: 100nF, Capacitor_SMD:C_0805_2012Metric_Pad1.18x1.45mm_HandSolder, B.Cu at (154.1, 89.1)
- added C18: 1uF, Capacitor_SMD:C_0805_2012Metric_Pad1.18x1.45mm_HandSolder, B.Cu at (141.6, 97.8)
- added J10: PROG_PORT, Connector_PinHeader_2.54mm:PinHeader_1x02_P2.54mm_Vertical, F.Cu at (142.0, 105.5)
- added J11: PROG_PORT, Connector_PinHeader_2.54mm:PinHeader_1x02_P2.54mm_Vertical, F.Cu at (149.1, 108.0)
- added J9: PROG_PORT, Connector_PinHeader_2.54mm:PinHeader_1x02_P2.54mm_Vertical, F.Cu at (144.8, 86.5)
- added R10: 20k, Resistor_SMD:R_0805_2012Metric_Pad1.20x1.40mm_HandSolder, F.Cu at (133.1, 94.6)
- added U20: BSD316, Package_TO_SOT_SMD:SOT-363_SC-70-6_Handsoldering, F.Cu at (138.6, 104.6)
- added U21: BSD316, Package_TO_SOT_SMD:SOT-363_SC-70-6_Handsoldering, F.Cu at (145.7, 104.3)
- added U22: W25Q40CL, Package_SO:SOIC-8W_5.3x5.3mm_P1.27mm, B.Cu at (150.2, 94.7)
- J4: value Serial -> PROG_PORT; footprint Connector_PinHeader_2.54mm:PinHeader_1x03_P2.54mm_Vertical -> Connector_PinHeader_2.54mm:PinHeader_1x02_P2.54mm_Vertical
- moved J7 86.3 mm to (101.8, 135.0), turned to 90 degrees
- moved R39 39.6 mm to (116.4, 114.7)
- moved R40 39.3 mm to (116.3, 110.4), turned to 180 degrees
- moved J5 36.7 mm to (137.3, 49.0)
- moved J4 32.0 mm to (142.2, 110.4), turned to 90 degrees
- moved R3 19.1 mm to (142.2, 100.1)
- moved R20 16.1 mm to (146.7, 116.7)
- moved TH1 16.0 mm to (142.1, 116.5)
- moved TH2 11.1 mm to (142.0, 125.8)
- moved R21 11.1 mm to (147.1, 125.9)
- moved C8 9.94 mm to (138.4, 100.2)
- moved J6 9.46 mm to (170.9, 102.2)
- moved C10 8.11 mm to (140.6, 91.5)
- moved C11 8.11 mm to (151.8, 98.2)
- moved C13 8.11 mm to (160.9, 98.5)
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Connections:
- net CELL_DSCHG_1 renamed /MCU/CELL_DSCHG_1_MCU
- net CELL_DSCHG_2 renamed /MCU/CELL_DSCHG_2_MCU
- net CELL_DSCHG_3 renamed /MCU/CELL_DSCHG_3_MCU
- net TEMP_SENSE_1 renamed /MCU/TEMP_SENSE_1
- net TEMP_SENSE_2 renamed /MCU/TEMP_SENSE_2
- net TEMP_SENSE_3 renamed /MCU/TEMP_SENSE_3
- net USB_PWR renamed VBUS
- J4 pad 1: RXD -> /MCU/EN
- J4 pad 2: TXD -> /MCU/IO0
- R22 pad 2: CELL_MEAS_3 -> /MCU/CELL_MEAS_3_MCU
- R23 pad 1: CELL_MEAS_3 -> /MCU/CELL_MEAS_3_MCU
- R26 pad 2: CELL_MEAS_2 -> /MCU/CELL_MEAS_2_MCU
- R27 pad 1: CELL_MEAS_2 -> /MCU/CELL_MEAS_2_MCU
- R28 pad 2: CELL_MEAS_1 -> /MCU/CELL_MEAS_1_MCU
- R29 pad 1: CELL_MEAS_1 -> /MCU/CELL_MEAS_1_MCU
- U1 pad 11: unconnected-(U1-Pad11) -> Net-(R39-Pad2)
- U1 pad 20: unconnected-(U1-Pad20) -> /MCU/CELL_MEAS_3_MCU
- U1 pad 21: unconnected-(U1-Pad21) -> /MCU/CELL_MEAS_2_MCU
- U1 pad 22: CELL_MEAS_3 -> /MCU/CELL_MEAS_1_MCU
- U1 pad 23: CELL_MEAS_2 -> /MCU/IO0
- U1 pad 24: CELL_MEAS_1 -> unconnected-(U1-Pad24)
- U1 pad 26: unconnected-(U1-Pad26) -> Net-(U1-Pad26)
- U1 pad 28: unconnected-(U1-Pad28) -> /MCU/SD_DATA_2
- U1 pad 29: unconnected-(U1-Pad29) -> /MCU/SD_DATA_3
- U1 pad 30: unconnected-(U1-Pad30) -> /MCU/SD_CMD
- U1 pad 31: unconnected-(U1-Pad31) -> /MCU/SD_CLK
- U1 pad 32: unconnected-(U1-Pad32) -> /MCU/SD_DATA_0
- U1 pad 33: unconnected-(U1-Pad33) -> /MCU/SD_DATA_1
- U1 pad 35: Net-(R39-Pad2) -> unconnected-(U1-Pad35)
- U1 pad 38: DRIVER_EN -> /MCU/DRIVER_DIR_MCU
- U1 pad 39: ~DRIVER_DIR -> /MCU/DRIVER_EN_MCU
- U1 pad 40: RXD -> /MCU/RXD_MCU
- U1 pad 41: TXD -> /MCU/TXD_MCU
- U1 pad 9: unconnected-(U1-Pad9) -> /MCU/EN
- U18 pad 3: DRIVER_EN -> /MCU/DRIVER_EN_MCU
- U2 pad 2: ~DRIVER_DIR -> /MCU/DRIVER_DIR_MCU
- U6 pad 2: ~DRIVER_DIR -> /MCU/DRIVER_DIR_MCU
- U6 pad 3: DRIVER_EN -> /MCU/DRIVER_EN_MCU
- U7 pad 2: ~DRIVER_DIR -> /MCU/DRIVER_DIR_MCU
Routing:
- net +3V3: track 0.58 -> 83.8 mm
- net PWR_UNREG: track 61.0 -> 134.9 mm
- net /MCU/CELL_MEAS_2_MCU: track 0.00 -> 69.7 mm
- net /MCU/CELL_MEAS_1_MCU: track 0.00 -> 68.1 mm
- net CELL_MEAS_2: track 66.7 -> 0.00 mm
- net CELL_MEAS_1: track 66.1 -> 0.00 mm
- net /MCU/CELL_MEAS_3_MCU: track 0.00 -> 64.0 mm
- net /MCU/DRIVER_EN_MCU: track 0.00 -> 60.9 mm, vias 0 -> 1
- net CELL_MEAS_3: track 59.8 -> 0.00 mm
- net DRIVER_EN: track 59.2 -> 0.00 mm, vias 3 -> 0
- net ~DRIVER_DIR: track 57.8 -> 0.00 mm, vias 1 -> 0
- net /MCU/DRIVER_DIR_MCU: track 0.00 -> 57.1 mm, vias 0 -> 1
- net VBUS: track 123.9 -> 69.0 mm, vias 4 -> 2
- net /MCU/3V3_MCU: track 13.2 -> 65.2 mm, vias 4 -> 6
- net /MCU/EN: track 0.00 -> 31.7 mm, vias 0 -> 2
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