File: schematic/MCU.kicad_sch (KiCad schematic)
At the start: 16 parts, among them U1 ESP32-D-WD-V3, Y1 Crystal_GND24

Commit message: prelim ble working
Changed lines of the file:
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@@
+    (stroke (width 0) (type default) (color 0 0 0 0))
+  )
+  (wire (pts (xy 97.79 101.6) (xy 149.86 101.6))
     (stroke (width 0) (type default) (color 0 0 0 0))
   )

Commit message: e
Parts:
- added R3: 0, Resistor_SMD:R_0805_2012Metric_Pad1.20x1.40mm_HandSolder, symbol Device:R
Connections:
- net +3V3 renamed 3V3_MCU
- net 3V3_MCU: now also R3.2
- net TURBO_EN: no longer names the net of U1.42 (GPIO21)
- new net 3V3: R3.1
Other:
- moved on the sheet: C8

Commit message: e
Parts:
- added C16, C17: 100nF, Capacitor_SMD:C_0805_2012Metric_Pad1.18x1.45mm_HandSolder, symbol Device:C
- added C18: 1uF, Capacitor_SMD:C_0805_2012Metric_Pad1.18x1.45mm_HandSolder, symbol Device:C
- added J10, J11, J4, J9: PROG_PORT, Connector_PinHeader_2.54mm:PinHeader_1x02_P2.54mm_Vertical, symbol Connector:Conn_01x02_Male
- added R10: 20k, Resistor_SMD:R_0805_2012Metric_Pad1.20x1.40mm_HandSolder, symbol Device:R
- added U20, U21: BSD316, Package_TO_SOT_SMD:SOT-363_SC-70-6_Handsoldering, symbol 1KicadLib:BSD316
- added U22: W25Q40CL, Package_SO:SOIC-8W_5.3x5.3mm_P1.27mm, symbol 1KicadLib:W25Q40CL
Connections:
- net ~DRIVER_DIR is gone; now on net DRIVER_EN: U1.39 (GPIO22)
- net 3V3_MCU: now also C17.1, J11.1 (Pin_1), R10.1, U22.8 (VCC)
- net DRIVER_EN: no longer U1.38 (GPIO19)
- net GND: now also C16.2, C17.2, C18.2, J11.2 (Pin_2), U22.4 (GND)
- net RXD: now also J9.1 (Pin_1)
- net TXD: now also J9.2 (Pin_2)
- net at U1.11 (GPIO35/VDET_2): now also R39.2, R40.1
- net CELL_3_VOLTAGE: now reaches U1.20 (GPIO13/MTCK)
- net CELL_2_VOLTAGE: now reaches U1.21 (GPIO15/MTDO)
- net at U1.26 (VDD_SDIO): now also C18.1
- net SD_DATA_2: now reaches U1.28 (SD_DATA_2)
- net SD_DATA_2: now also U22.7 (~{HOLD})
- net SD_DATA_3: now reaches U1.29 (SD_DATA_3)
- net SD_DATA_3: now also U22.3 (~{WP})
- net SD_CMD: now reaches U1.30 (SD_CMD)
- net SD_CMD: now also U22.1 (~{CS})
- net SD_CLK: now reaches U1.31 (SD_CLK)
- net SD_CLK: now also U22.6 (CLK)
- net SD_DATA_0: now reaches U1.32 (SD_DATA_0)
- net SD_DATA_0: now also U22.2 (DO)
- net SD_DATA_1: now reaches U1.33 (SD_DATA_1)
- net SD_DATA_1: now also U22.5 (DI)
- net EN: now reaches U1.9 (CHIP_PU)
- net EN: now also C16.1, J4.1 (Pin_1), R10.2, U20.1 (D), U20.2 (D), U20.5 (D), U20.6 (D)
- net CELL_DSCHG_1 renamed CELL_1_DSCHG
- net CELL_DSCHG_2 renamed CELL_2_DSCHG
- net CELL_DSCHG_3 renamed CELL_3_DSCHG
- net CELL_MEAS_1: no longer names the net of U1.24 (GPIO4)
- net CELL_MEAS_2 renamed IO0
- net IO0: now also J4.2 (Pin_2), U21.1 (D), U21.2 (D), U21.5 (D), U21.6 (D)
- net CELL_MEAS_3 renamed CELL_1_VOLTAGE
- net USB_PWR renamed USB_AVAIL_DETECT
- new net DRIVER_DIR: U1.38 (GPIO19)
- new net DTR: J10.1 (Pin_1), U20.3 (G), U21.4 (S)
- new net RTS: J10.2 (Pin_2), U20.4 (S), U21.3 (G)
- now unconnected: U1.35 (GPIO18)
Other:
- note added: "1.375 track width .25 clearance for waveguide"
- note removed: "1.375 track width .25 clearance"
- moved on the sheet: C8, R3, R39, R40
