File: schematic/pwrmngmt.kicad_sch (KiCad schematic)
At the start: 55 parts, among them U10 BSD316, U11 BSD316, U12 PC817, U13 PC817, U14 PC817, U15 AS431, U16 NL17SZ14, U17 XL6009, U19 XC9247B75CMR-G, U20 MIC5211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

Commit message: e
Parts:
- removed C16, C17: 100nF, Capacitor_SMD:C_0805_2012Metric_Pad1.18x1.45mm_HandSolder, symbol Device:C
- removed C19: 10uF, Capacitor_SMD:C_0805_2012Metric_Pad1.18x1.45mm_HandSolder, symbol Device:C
- removed C22: 1uF, Capacitor_SMD:C_0805_2012Metric_Pad1.18x1.45mm_HandSolder, symbol Device:C
- removed D3: LL4148, Diode_SMD:D_MiniMELF, symbol Diode:LL4148
- removed D5: PMEG40T20EPX, Diode_SMD:D_SOD-128, symbol Device:D_Schottky
- removed R10: 27k, Resistor_SMD:R_0805_2012Metric_Pad1.20x1.40mm_HandSolder, symbol Device:R
- removed R2: 300k, Resistor_SMD:R_0805_2012Metric_Pad1.20x1.40mm_HandSolder, symbol Device:R
- removed R3: 62k, Resistor_SMD:R_0805_2012Metric_Pad1.20x1.40mm_HandSolder, symbol Device:R
- removed U16: NL17SZ14, Package_TO_SOT_SMD:SOT-553, symbol 1KicadLib:NL17SZ14
- removed U19: XC9247B75CMR-G, Package_TO_SOT_SMD:SOT-23-6_Handsoldering, symbol 1KicadLib:XC9247B75CMR-G
- removed U20: MIC5211, Package_TO_SOT_SMD:SOT-23-6_Handsoldering, symbol 1KicadLib:MIC5211
- added U16: AP63203WU, Package_TO_SOT_SMD:TSOT-23-6, symbol Regulator_Switching:AP63203WU
- added U19: HT75xx-1-SOT89, Package_TO_SOT_SMD:SOT-89-3, symbol Regulator_Linear:HT75xx-1-SOT89
- C11: value 2.2uF -> 100nF
- C12: value 100uF -> 10uF; footprint Capacitor_SMD:C_1210_3225Metric_Pad1.33x2.70mm_HandSolder -> Capacitor_SMD:C_0805_2012Metric_Pad1.18x1.45mm_HandSolder
- C13: value 100uF -> 22uF; footprint Capacitor_SMD:C_1210_3225Metric_Pad1.33x2.70mm_HandSolder -> Capacitor_SMD:C_0805_2012Metric_Pad1.18x1.45mm_HandSolder
- C14: value 130pF -> 22uF
- C9: value 1uF -> 10uF
Connections:
- net GND: now also C14.2, U16.4 (GND), U19.1 (GND)
- net PWR_UNREG: now also C9.1, U16.2 (EN), U16.3 (IN), U19.2 (VIN)
- net at L2.1: now also C11.1, U16.5 (SW); no longer C11.2
- net +3V3 renamed 3V3
- net 3V3: now also U16.1 (FB); no longer C12.1
- new net: C11.2, U16.6 (BST)
- new net 5V: C12.1, U19.3 (VOUT)
Other:
- note added: "5V Linear"
- note removed: "3.3V Linear, 5V Linear"
