File: schematic/pwrmngmt.kicad_sch (KiCad schematic)
At the start: 45 parts, among them U10 BSD316, U11 BSD316, U12 PC817, U13 PC817, U14 PC817, U15 AS431, U16 AP63203WU, U17 XL6009, U19 HT75xx-1-SOT89, U5 LM324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

Commit message: E
Connections:
- net +BATT renamed PWR_SW_P
- net PWR_UNREG renamed VCC_UNREGULATED
Changed lines of the file:
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@@
     (stroke (width 0) (type default) (color 0 0 0 0))
   )
-  (wire (pts (xy 204.47 82.55) (xy 204.47 83.82))
+  (wire (pts (xy 204.47 74.93) (xy 204.47 83.82))
     (stroke (width 0) (type default) (color 0 0 0 0))
   )
@@
     (stroke (width 0) (type default) (color 0 0 0 0))
   )
-  (wire (pts (xy 185.42 31.75) (xy 185.42 33.02))
+  (wire (pts (xy 185.42 24.13) (xy 185.42 33.02))
     (stroke (width 0) (type default) (color 0 0 0 0))
   )
@@
     (stroke (width 0) (type default) (color 0 0 0 0))
   )
-  (wire (pts (xy 156.21 31.75) (xy 165.1 31.75))
+  (wire (pts (xy 156.21 31.75) (xy 158.75 31.75))
     (stroke (width 0) (type default) (color 0 0 0 0))
   )
@@
     (effects (font (size 3 3)) (justify left bottom))
   )
+  (label "PWR__UNREG_PWRMG" (at 158.75 31.75 0)
+    (effects (font (size 1.27 1.27)) (justify left bottom))
+  )
+  (label "BATT" (at 21.59 20.32 0)
+    (effects (font (size 1.27 1.27)) (justify left bottom))
+  )
+  (label "PWR__UNREG_PWRMG" (at 185.42 24.13 0)
+    (effects (font (size 1.27 1.27)) (justify left bottom))
+  )
+  (label "BATT" (at 21.59 142.24 0)
+    (effects (font (size 1.27 1.27)) (justify left bottom))
+  )
+  (label "BATT" (at 142.24 140.97 0)
+    (effects (font (size 1.27 1.27)) (justify left bottom))
+  )
+  (label "PWR__UNREG_PWRMG" (at 204.47 74.93 0)
+    (effects (font (size 1.27 1.27)) (justify left bottom))
+  )
   (label "5V" (at 160.02 45.72 0)
     (effects (font (size 1.27 1.27)) (justify left bottom))
   )
   (label "3V3" (at 264.16 30.48 0)
+    (effects (font (size 1.27 1.27)) (justify left bottom))
+  )
+  (label "BATT" (at 161.29 25.4 0)
     (effects (font (size 1.27 1.27)) (justify left bottom))
   )
@@
     (pin "2")
   )
-  (symbol (lib_id "1KicadPowerLib:PWR_UNREG") (at 165.1 30.48 0) (unit 1)
-    (in_bom yes) (on_board yes) (fields_autoplaced)
-    (property "Reference" "#PWR_UNREG0106" (id 0) (at 160.655 31.115 0)
-      (effects (font (size 1.27 1.27)) hide)
-    )
-    (property "Value" "PWR_UNREG" (id 1) (at 165.1 28.098 0))
-    (property "Footprint" "" (id 2) (at 168.91 31.75 0)
-      (effects (font (size 1.27 1.27)) hide)
-    )
-    (property "Datasheet" "" (id 3) (at 168.91 31.75 0)
-      (effects (font (size 1.27 1.27)) hide)
-    )
-    (pin "1")
-  )
   (symbol (lib_id "Device:R") (at 105.41 59.69 0) (unit 1)
     (in_bom yes) (on_board yes) (fields_autoplaced)
@@
     (pin "1")
     (pin "2")
-  )
-  (symbol (lib_name "PWR_UNREG_2") (lib_id "1KicadPowerLib:PWR_UNREG") (at 204.47 81.28 0) (unit 1)
-    (in_bom yes) (on_board yes) (fields_autoplaced)
-    (property "Reference" "#PWR_UNREG0102" (id 0) (at 200.025 81.915 0)
-      (effects (font (size 1.27 1.27)) hide)
-    )
-    (property "Value" "PWR_UNREG" (id 1) (at 204.47 78.898 0))
-    (property "Footprint" "" (id 2) (at 208.28 82.55 0)
-      (effects (font (size 1.27 1.27)) hide)
-    )
-    (property "Datasheet" "" (id 3) (at 208.28 82.55 0)
-      (effects (font (size 1.27 1.27)) hide)
-    )
-    (pin "1")
   )
   (symbol (lib_id "Regulator_Switching:AP63203WU") (at 199.39 35.56 0) (unit 1)
@@
     (pin "2")
   )
-  (symbol (lib_id "power:+BATT") (at 21.59 142.24 0) (unit 1)
-    (in_bom yes) (on_board yes) (fields_autoplaced)
-    (property "Reference" "#PWR0169" (id 0) (at 21.59 146.05 0)
-      (effects (font (size 1.27 1.27)) hide)
-    )
-    (property "Value" "+BATT" (id 1) (at 21.59 138.6642 0))
-    (property "Footprint" "" (id 2) (at 21.59 142.24 0)
-      (effects (font (size 1.27 1.27)) hide)
-    )
-    (property "Datasheet" "" (id 3) (at 21.59 142.24 0)
-      (effects (font (size 1.27 1.27)) hide)
-    )
-    (pin "1")
-  )
   (symbol (lib_id "Device:R") (at 102.87 36.83 0) (unit 1)
     (in_bom yes) (on_board yes) (fields_autoplaced)
@@
     (pin "1")
     (pin "2")
-  )
-  (symbol (lib_name "PWR_UNREG_2") (lib_id "1KicadPowerLib:PWR_UNREG") (at 185.42 30.48 0) (unit 1)
-    (in_bom yes) (on_board yes) (fields_autoplaced)
-    (property "Reference" "#PWR_UNREG0101" (id 0) (at 180.975 31.115 0)
-      (effects (font (size 1.27 1.27)) hide)
-    )
-    (property "Value" "PWR_UNREG" (id 1) (at 185.42 28.098 0))
-    (property "Footprint" "" (id 2) (at 189.23 31.75 0)
-      (effects (font (size 1.27 1.27)) hide)
-    )
-    (property "Datasheet" "" (id 3) (at 189.23 31.75 0)
-      (effects (font (size 1.27 1.27)) hide)
-    )
-    (pin "1")
   )
   (symbol (lib_id "Device:R") (at 45.72 124.46 270) (unit 1)
@@
     (pin "2")
   )
-  (symbol (lib_id "power:+BATT") (at 142.24 140.97 0) (unit 1)
-    (in_bom yes) (on_board yes) (fields_autoplaced)
-    (property "Reference" "#PWR0145" (id 0) (at 142.24 144.78 0)
-      (effects (font (size 1.27 1.27)) hide)
-    )
-    (property "Value" "+BATT" (id 1) (at 142.24 137.3942 0))
-    (property "Footprint" "" (id 2) (at 142.24 140.97 0)
-      (effects (font (size 1.27 1.27)) hide)
-    )
-    (property "Datasheet" "" (id 3) (at 142.24 140.97 0)
-      (effects (font (size 1.27 1.27)) hide)
-    )
-    (pin "1")
-  )
   (symbol (lib_id "Device:R") (at 21.59 160.02 0) (unit 1)
     (in_bom yes) (on_board yes) (fields_autoplaced)
@@
       (effects (font (size 1.27 1.27)) hide)
     )
-    (pin "1")
-  )
-  (symbol (lib_id "power:+BATT") (at 161.29 25.4 0) (unit 1)
-    (in_bom yes) (on_board yes) (fields_autoplaced)
-    (property "Reference" "#PWR0163" (id 0) (at 161.29 29.21 0)
-      (effects (font (size 1.27 1.27)) hide)
-    )
-    (property "Value" "+BATT" (id 1) (at 161.29 21.8242 0))
-    (property "Footprint" "" (id 2) (at 161.29 25.4 0)
-      (effects (font (size 1.27 1.27)) hide)
-    )
-    (property "Datasheet" "" (id 3) (at 161.29 25.4 0)
-      (effects (font (size 1.27 1.27)) hide)
-    )
-    (pin "1")
-  )
-  (symbol (lib_id "power:+BATT") (at 21.59 20.32 0) (unit 1)
-    (in_bom yes) (on_board yes) (fields_autoplaced)
-    (property "Reference" "#PWR0175" (id 0) (at 21.59 24.13 0)
-      (effects (font (size 1.27 1.27)) hide)
-    )
-    (property "Value" "+BATT" (id 1) (at 21.59 16.7442 0))
-    (property "Footprint" "" (id 2) (at 21.59 20.32 0)
-      (effects (font (size 1.27 1.27)) hide)
-    )
-    (property "Datasheet" "" (id 3) (at 21.59 20.32 0)
-      (effects (font (size 1.27 1.27)) hide)
-    )
