File: schematic/driver.kicad_sch (KiCad schematic)
At the start: 8 parts, among them J1 Peltier Connection, U18 slg55021, U2 NL17SZ14, U3 DMT3020LSDQ, U4 DMT3020LSDQ, U6 slg55021, U7 NL17SZ14, U8 NL17SZ14

Commit message: e
Parts:
- added R2: 0, Resistor_SMD:R_0805_2012Metric_Pad1.20x1.40mm_HandSolder, symbol Device:R
Connections:
- net +5V renamed 5V_PD
- net 5V_PD: now also R2.2
- net PWR_UNREG renamed VCC_UNREGULATED
- new net 5V: R2.1
Changed lines of the file:
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@@
     (stroke (width 0) (type default) (color 0 0 0 0))
   )
-  (wire (pts (xy 217.17 87.63) (xy 217.17 86.36))
+  (wire (pts (xy 217.17 85.09) (xy 217.17 87.63))
     (stroke (width 0) (type default) (color 0 0 0 0))
   )
@@
     (stroke (width 0) (type default) (color 0 0 0 0))
   )
-  (wire (pts (xy 81.28 87.63) (xy 81.28 86.36))
-    (stroke (width 0) (type default) (color 0 0 0 0))
-  )
   (wire (pts (xy 100.33 90.17) (xy 118.11 90.17))
     (stroke (width 0) (type default) (color 0 0 0 0))
@@
     (stroke (width 0) (type default) (color 0 0 0 0))
   )
+  (wire (pts (xy 199.39 102.87) (xy 199.39 105.41))
+    (stroke (width 0) (type default) (color 0 0 0 0))
+  )
   (wire (pts (xy 144.78 100.33) (xy 144.78 142.24))
     (stroke (width 0) (type default) (color 0 0 0 0))
@@
     (stroke (width 0) (type default) (color 0 0 0 0))
   )
+  (wire (pts (xy 133.35 170.18) (xy 140.97 170.18))
+    (stroke (width 0) (type default) (color 0 0 0 0))
+  )
   (wire (pts (xy 172.72 121.92) (xy 172.72 116.84))
     (stroke (width 0) (type default) (color 0 0 0 0))
@@
     (stroke (width 0) (type default) (color 0 0 0 0))
   )
+  (wire (pts (xy 77.47 85.09) (xy 77.47 87.63))
+    (stroke (width 0) (type default) (color 0 0 0 0))
+  )
   (wire (pts (xy 116.84 151.13) (xy 116.84 148.59))
     (stroke (width 0) (type default) (color 0 0 0 0))
@@
     (stroke (width 0) (type default) (color 0 0 0 0))
   )
-  (wire (pts (xy 82.55 87.63) (xy 81.28 87.63))
+  (wire (pts (xy 77.47 87.63) (xy 82.55 87.63))
     (stroke (width 0) (type default) (color 0 0 0 0))
   )
@@
     (stroke (width 0) (type default) (color 0 0 0 0))
   )
+  (wire (pts (xy 250.19 78.74) (xy 250.19 81.28))
+    (stroke (width 0) (type default) (color 0 0 0 0))
+  )
   (wire (pts (xy 100.33 92.71) (xy 119.38 92.71))
     (stroke (width 0) (type default) (color 0 0 0 0))
@@
     (stroke (width 0) (type default) (color 0 0 0 0))
   )
-  (wire (pts (xy 107.95 170.18) (xy 116.84 170.18))
+  (wire (pts (xy 107.95 170.18) (xy 125.73 170.18))
     (stroke (width 0) (type default) (color 0 0 0 0))
   )
@@
     (stroke (width 0) (type default) (color 0 0 0 0))
   )
+  (wire (pts (xy 104.14 106.68) (xy 104.14 109.22))
+    (stroke (width 0) (type default) (color 0 0 0 0))
+  )
   (wire (pts (xy 172.72 100.33) (xy 172.72 99.06))
     (stroke (width 0) (type default) (color 0 0 0 0))
+  )
+  (label "5V_PD" (at 250.19 78.74 0)
+    (effects (font (size 1.27 1.27)) (justify left bottom))
+  )
+  (label "PWR_UNREG_PD" (at 116.84 148.59 0)
+    (effects (font (size 1.27 1.27)) (justify left bottom))
+  )
+  (label "5V_PD" (at 104.14 106.68 0)
+    (effects (font (size 1.27 1.27)) (justify left bottom))
+  )
+  (label "5V_PD" (at 77.47 85.09 0)
+    (effects (font (size 1.27 1.27)) (justify left bottom))
+  )
+  (label "5V_PD" (at 217.17 85.09 0)
+    (effects (font (size 1.27 1.27)) (justify left bottom))
+  )
+  (label "5V_PD" (at 140.97 170.18 0)
+    (effects (font (size 1.27 1.27)) (justify left bottom))
+  )
+  (label "5V_PD" (at 199.39 102.87 0)
+    (effects (font (size 1.27 1.27)) (justify left bottom))
+  )
+  (label "PWR_UNREG_PD" (at 151.13 72.39 0)
+    (effects (font (size 1.27 1.27)) (justify left bottom))
   )
   (global_label "~DRIVER_DIR" (shape input) (at 260.35 90.17 0) (fields_autoplaced)
@@
     (pin "1")
   )
-  (symbol (lib_id "power:+5V") (at 199.39 105.41 0) (unit 1)
-    (in_bom yes) (on_board yes) (fields_autoplaced)
-    (property "Reference" "#PWR0133" (id 0) (at 199.39 109.22 0)
-      (effects (font (size 1.27 1.27)) hide)
-    )
-    (property "Value" "+5V" (id 1) (at 199.39 101.8342 0))
-    (property "Footprint" "" (id 2) (at 199.39 105.41 0)
-      (effects (font (size 1.27 1.27)) hide)
-    )
-    (property "Datasheet" "" (id 3) (at 199.39 105.41 0)
-      (effects (font (size 1.27 1.27)) hide)
-    )
-    (pin "1")
-  )
-  (symbol (lib_id "1KicadPowerLib:PWR_UNREG") (at 151.13 71.12 0) (unit 1)
-    (in_bom yes) (on_board yes) (fields_autoplaced)
-    (property "Reference" "#PWR_UNREG0104" (id 0) (at 146.685 71.755 0)
-      (effects (font (size 1.27 1.27)) hide)
-    )
-    (property "Value" "PWR_UNREG" (id 1) (at 151.13 68.738 0))
-    (property "Footprint" "" (id 2) (at 154.94 72.39 0)
-      (effects (font (size 1.27 1.27)) hide)
-    )
-    (property "Datasheet" "" (id 3) (at 154.94 72.39 0)
-      (effects (font (size 1.27 1.27)) hide)
-    )
-    (pin "1")
-  )
   (symbol (lib_id "Connector:Conn_01x02_Female") (at 165.1 139.7 0) (unit 1)
     (in_bom yes) (on_board yes)
@@
     )
     (property "Datasheet" "~" (id 3) (at 165.1 139.7 0)
+      (effects (font (size 1.27 1.27)) hide)
+    )
+    (pin "1")
+    (pin "2")
+  )
+  (symbol (lib_id "Device:R") (at 129.54 170.18 90) (unit 1)
+    (in_bom yes) (on_board yes) (fields_autoplaced)
+    (property "Reference" "R2" (id 0) (at 129.54 165.4642 90))
+    (property "Value" "0" (id 1) (at 129.54 168.0011 90))
+    (property "Footprint" "Resistor_SMD:R_0805_2012Metric_Pad1.20x1.40mm_HandSolder" (id 2) (at 129.54 171.958 90)
+      (effects (font (size 1.27 1.27)) hide)
+    )
+    (property "Datasheet" "~" (id 3) (at 129.54 170.18 0)
       (effects (font (size 1.27 1.27)) hide)
     )
@@
     (pin "5")
   )
-  (symbol (lib_id "power:+5V") (at 250.19 81.28 0) (mirror y) (unit 1)
-    (in_bom yes) (on_board yes) (fields_autoplaced)
-    (property "Reference" "#PWR0121" (id 0) (at 250.19 85.09 0)
-      (effects (font (size 1.27 1.27)) hide)
-    )
-    (property "Value" "+5V" (id 1) (at 250.19 77.7042 0))
-    (property "Footprint" "" (id 2) (at 250.19 81.28 0)
-      (effects (font (size 1.27 1.27)) hide)
-    )
-    (property "Datasheet" "" (id 3) (at 250.19 81.28 0)
-      (effects (font (size 1.27 1.27)) hide)
-    )
-    (pin "1")
-  )
-  (symbol (lib_id "power:+5V") (at 104.14 109.22 0) (unit 1)
-    (in_bom yes) (on_board yes) (fields_autoplaced)
-    (property "Reference" "#PWR0131" (id 0) (at 104.14 113.03 0)
-      (effects (font (size 1.27 1.27)) hide)
-    )
-    (property "Value" "+5V" (id 1) (at 104.14 105.6442 0))
-    (property "Footprint" "" (id 2) (at 104.14 109.22 0)
-      (effects (font (size 1.27 1.27)) hide)
-    )
-    (property "Datasheet" "" (id 3) (at 104.14 109.22 0)
-      (effects (font (size 1.27 1.27)) hide)
-    )
-    (pin "1")
-  )
   (symbol (lib_id "1KicadLib:DMT3020LSDQ") (at 127 90.17 0) (unit 1)
     (in_bom yes) (on_board yes) (fields_autoplaced)
@@
     (pin "7")
     (pin "8")
-  )
-  (symbol (lib_name "PWR_UNREG_1") (lib_id "1KicadPowerLib:PWR_UNREG") (at 116.84 147.32 0) (unit 1)
-    (in_bom yes) (on_board yes) (fields_autoplaced)
-    (property "Reference" "#PWR_UNREG0105" (id 0) (at 112.395 147.955 0)
-      (effects (font (size 1.27 1.27)) hide)
-    )
-    (property "Value" "PWR_UNREG" (id 1) (at 116.84 144.938 0))
-    (property "Footprint" "" (id 2) (at 120.65 148.59 0)
-      (effects (font (size 1.27 1.27)) hide)
-    )
-    (property "Datasheet" "" (id 3) (at 120.65 148.59 0)
-      (effects (font (size 1.27 1.27)) hide)
-    )
-    (pin "1")
   )
   (symbol (lib_id "power:GND") (at 81.28 96.52 0) (unit 1)
@@
     )
     (property "Datasheet" "" (id 3) (at 104.14 127 0)
-      (effects (font (size 1.27 1.27)) hide)
-    )
-    (pin "1")
-  )
-  (symbol (lib_id "power:+5V") (at 217.17 86.36 0) (mirror y) (unit 1)
-    (in_bom yes) (on_board yes) (fields_autoplaced)
-    (property "Reference" "#PWR0135" (id 0) (at 217.17 90.17 0)
-      (effects (font (size 1.27 1.27)) hide)
-    )
-    (property "Value" "+5V" (id 1) (at 217.17 82.7842 0))
-    (property "Footprint" "" (id 2) (at 217.17 86.36 0)
-      (effects (font (size 1.27 1.27)) hide)
-    )
-    (property "Datasheet" "" (id 3) (at 217.17 86.36 0)
       (effects (font (size 1.27 1.27)) hide)
     )
@@
     (pin "8")
   )
-  (symbol (lib_id "power:+5V") (at 81.28 86.36 0) (unit 1)
-    (in_bom yes) (on_board yes) (fields_autoplaced)
-    (property "Reference" "#PWR0120" (id 0) (at 81.28 90.17 0)
-      (effects (font (size 1.27 1.27)) hide)
-    )
-    (property "Value" "+5V" (id 1) (at 81.28 82.7842 0))
-    (property "Footprint" "" (id 2) (at 81.28 86.36 0)
-      (effects (font (size 1.27 1.27)) hide)
-    )
-    (property "Datasheet" "" (id 3) (at 81.28 86.36 0)
-      (effects (font (size 1.27 1.27)) hide)
-    )
-    (pin "1")
-  )
-  (symbol (lib_id "power:+5V") (at 116.84 170.18 0) (unit 1)
-    (in_bom yes) (on_board yes) (fields_autoplaced)
-    (property "Reference" "#PWR0132" (id 0) (at 116.84 173.99 0)
-      (effects (font (size 1.27 1.27)) hide)
-    )
-    (property "Value" "+5V" (id 1) (at 116.84 166.6042 0))
-    (property "Footprint" "" (id 2) (at 116.84 170.18 0)
-      (effects (font (size 1.27 1.27)) hide)
-    )
-    (property "Datasheet" "" (id 3) (at 116.84 170.18 0)
-      (effects (font (size 1.27 1.27)) hide)
-    )
-    (pin "1")
-  )
   (symbol (lib_id "1KicadLib:NL17SZ14") (at 102.87 118.11 0) (unit 1)

Commit message: e
Connections:
- net ~DRIVER_DIR renamed DRIVER_DIR
Changed lines of the file:
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@@
+    (effects (font (size 1.27 1.27)) (justify left bottom))
+  )
+  (label "DRIVER_DIR_PD" (at 115.57 156.21 0)
     (effects (font (size 1.27 1.27)) (justify left bottom))
   )
@@
     (effects (font (size 1.27 1.27)) (justify left bottom))
   )
+  (label "DRIVER_EN_PD" (at 78.74 92.71 180)
+    (effects (font (size 1.27 1.27)) (justify right bottom))
+  )
   (label "5V_PD" (at 104.14 106.68 0)
     (effects (font (size 1.27 1.27)) (justify left bottom))
   )
+  (label "DRIVER_EN_PD" (at 115.57 162.56 0)
+    (effects (font (size 1.27 1.27)) (justify left bottom))
+  )
+  (label "DRIVER_DIR_PD" (at 260.35 90.17 0)
+    (effects (font (size 1.27 1.27)) (justify left bottom))
+  )
+  (label "DRIVER_EN_PD" (at 217.17 92.71 0)
+    (effects (font (size 1.27 1.27)) (justify left bottom))
+  )
+  (label "DRIVER_DIR_PD" (at 91.44 118.11 180)
+    (effects (font (size 1.27 1.27)) (justify right bottom))
+  )
   (label "5V_PD" (at 77.47 85.09 0)
     (effects (font (size 1.27 1.27)) (justify left bottom))
+  )
+  (label "DRIVER_DIR_PD" (at 78.74 90.17 180)
+    (effects (font (size 1.27 1.27)) (justify right bottom))
   )
   (label "5V_PD" (at 217.17 85.09 0)
@@
     (effects (font (size 1.27 1.27)) (justify left bottom))
   )
-  (global_label "~DRIVER_DIR" (shape input) (at 260.35 90.17 0) (fields_autoplaced)
-    (effects (font (size 1.27 1.27)) (justify left))
-    (property "Intersheet References" "${INTERSHEET_REFS}" (id 0) (at 274.3461 90.0906 0)
-      (effects (font (size 1.27 1.27)) (justify left) hide)
-    )
-  )
-  (global_label "~DRIVER_DIR" (shape input) (at 115.57 156.21 0) (fields_autoplaced)
-    (effects (font (size 1.27 1.27)) (justify left))
-    (property "Intersheet References" "${INTERSHEET_REFS}" (id 0) (at 129.5661 156.2894 0)
-      (effects (font (size 1.27 1.27)) (justify left) hide)
-    )
-  )
-  (global_label "~DRIVER_DIR" (shape input) (at 91.44 118.11 180) (fields_autoplaced)
-    (effects (font (size 1.27 1.27)) (justify right))
-    (property "Intersheet References" "${INTERSHEET_REFS}" (id 0) (at 77.4439 118.0306 0)
-      (effects (font (size 1.27 1.27)) (justify right) hide)
-    )
-  )
-  (global_label "DRIVER_EN" (shape input) (at 78.74 92.71 180) (fields_autoplaced)
-    (effects (font (size 1.27 1.27)) (justify right))
-    (property "Intersheet References" "${INTERSHEET_REFS}" (id 0) (at 66.3163 92.6306 0)
-      (effects (font (size 1.27 1.27)) (justify right) hide)
-    )
-  )
-  (global_label "DRIVER_EN" (shape input) (at 217.17 92.71 0) (fields_autoplaced)
-    (effects (font (size 1.27 1.27)) (justify left))
-    (property "Intersheet References" "${INTERSHEET_REFS}" (id 0) (at 229.5937 92.6306 0)
-      (effects (font (size 1.27 1.27)) (justify left) hide)
-    )
-  )
-  (global_label "DRIVER_EN" (shape input) (at 115.57 162.56 0) (fields_autoplaced)
-    (effects (font (size 1.27 1.27)) (justify left))
-    (property "Intersheet References" "${INTERSHEET_REFS}" (id 0) (at 127.9937 162.4806 0)
-      (effects (font (size 1.27 1.27)) (justify left) hide)
-    )
-  )
-  (global_label "~DRIVER_DIR" (shape input) (at 78.74 90.17 180) (fields_autoplaced)
-    (effects (font (size 1.27 1.27)) (justify right))
-    (property "Intersheet References" "${INTERSHEET_REFS}" (id 0) (at 64.7439 90.0906 0)
-      (effects (font (size 1.27 1.27)) (justify right) hide)
-    )
-  )
   (hierarchical_label "5V" (shape input) (at 107.95 170.18 180)
     (effects (font (size 1.27 1.27)) (justify right))
@@
     (effects (font (size 1.27 1.27)) (justify right))
   )
-  (hierarchical_label "~DRIVER_DIR" (shape input) (at 107.95 156.21 180)
+  (hierarchical_label "DRIVER_DIR" (shape input) (at 107.95 156.21 180)
     (effects (font (size 1.27 1.27)) (justify right))
   )
