File: ProofOfConcepts/ChargerPOC/ChargerPOC/ChargerPOC.kicad_sch (KiCad schematic)
At the start: 48 parts, among them J1 PWM_VDRIVE_EN, J2 CELL_BAL_DISCH_EN, J3 CELL_MON_ADC, J4 USB_C_Receptacle_USB2.0, U10 LM324, U11 XL6009, U9 AS431

Commit message: E
Parts:
- removed C1, C2: 10uF, Capacitor_SMD:C_0805_2012Metric_Pad1.18x1.45mm_HandSolder, symbol Device:C
- removed D1, D2: LL4148, Diode_SMD:D_MiniMELF, symbol Diode:LL4148
- removed J1: PWM_VDRIVE_EN, Connector_PinHeader_2.54mm:PinHeader_1x02_P2.54mm_Vertical, symbol Connector:Conn_01x02_Male
- removed J4: USB_C_Receptacle_USB2.0, 1KicadLib:USB4125-GF-A, symbol 1KicadLib:USB_C_PWR_ONLY
- removed R12, R13: 5.1k, Capacitor_SMD:C_0805_2012Metric_Pad1.18x1.45mm_HandSolder, symbol Device:R
- added J1: VIN, 1KicadLib:GatorTestpoint, symbol Connector:Conn_01x01_Male
- added J4: CHG_CURR_MEAS_2, 1KicadLib:GatorTestpoint, symbol Connector:Conn_01x01_Male
- added J5: CHG_CURR_MEAS_1, 1KicadLib:GatorTestpoint, symbol Connector:Conn_01x01_Male
- added J6: GATOR_DIRT, 1KicadLib:GatorTestpoint, symbol Connector:Conn_01x01_Male
- J2, J3: footprint Connector_PinHeader_2.54mm:PinHeader_1x05_P2.54mm_Vertical -> Connector_PinHeader_2.54mm:PinHeader_1x04_P2.54mm_Vertical; symbol Connector:Conn_01x05_Male -> Connector:Conn_01x04_Male
- gave numbers to parts that had none: 22
Connections:
- net +BATT: now also J4.1 (Pin_1); no longer BT1.1 (+), R1.1, R7.1
- net GND: now also J6.1 (Pin_1)
- net VBUS: now also J1.1 (Pin_1)
- net at BT2.2 (-), BT3.1 (+), R22.1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: now also U6.4
- net at BT1.2 (-), BT2.1 (+), R2.1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: now also U5.4
- removed net Vdrive: U4.4, U5.4, U6.4
- new net: BT1.1 (+), J5.1 (Pin_1), R1.1, R7.1, U4.4

Commit message: e
Parts:
- removed R14: .1, Resistor_SMD:R_1206_3216Metric_Pad1.30x1.75mm_HandSolder, symbol Device:R
- added R?: .1, Resistor_SMD:R_1206_3216Metric_Pad1.30x1.75mm_HandSolder, symbol Device:R
- D3: footprint Diode_SMD:D_SMC_Handsoldering -> Diode_SMD:D_SMA_Handsoldering
- L1: footprint Inductor_SMD:L_12x12mm_H4.5mm -> Inductor_SMD:L_10.4x10.4_H4.8
- R10: value 18k -> 12k
- R9: value 100k -> 47k
- U9: footprint Package_TO_SOT_SMD:SOT-23-5_HandSoldering -> Package_TO_SOT_SMD:SOT-23
Connections:
- net GND: now also R?.2
Changed lines of the file:
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@@
+    (stroke (width 0) (type default) (color 0 0 0 0))
+  )
+  (wire (pts (xy 205.74 93.98) (xy 208.28 93.98))
     (stroke (width 0) (type default) (color 0 0 0 0))
   )
@@
   )
   (wire (pts (xy 97.79 92.71) (xy 97.79 95.25))
-    (stroke (width 0) (type default) (color 0 0 0 0))
-  )
-  (wire (pts (xy 198.12 91.44) (xy 200.66 91.44))
     (stroke (width 0) (type default) (color 0 0 0 0))
   )
@@
     (pin "2")
   )
-  (symbol (lib_id "power:GND") (at 200.66 91.44 0) (unit 1)
-    (in_bom yes) (on_board yes) (fields_autoplaced)
-    (property "Reference" "#PWR0104" (id 0) (at 200.66 97.79 0)
-      (effects (font (size 1.27 1.27)) hide)
-    )
-    (property "Value" "GND" (id 1) (at 200.66 95.8834 0))
-    (property "Footprint" "" (id 2) (at 200.66 91.44 0)
-      (effects (font (size 1.27 1.27)) hide)
-    )
-    (property "Datasheet" "" (id 3) (at 200.66 91.44 0)
-      (effects (font (size 1.27 1.27)) hide)
-    )
-    (pin "1")
-  )
   (symbol (lib_id "power:VBUS") (at 247.65 48.26 0) (unit 1)
     (in_bom yes) (on_board yes) (fields_autoplaced)
@@
     (property "Reference" "D3" (id 0) (at 198.4375 72.5002 0))
     (property "Value" "SS34" (id 1) (at 198.4375 75.0371 0))
-    (property "Footprint" "Diode_SMD:D_SMC_Handsoldering" (id 2) (at 198.12 77.47 0)
+    (property "Footprint" "Diode_SMD:D_SMA_Handsoldering" (id 2) (at 198.12 77.47 0)
       (effects (font (size 1.27 1.27)) hide)
     )
@@
       (effects (font (size 1.27 1.27)) (justify left))
     )
-    (property "Footprint" "Package_TO_SOT_SMD:SOT-23-5_HandSoldering" (id 2) (at 144.78 104.14 90)
+    (property "Footprint" "Package_TO_SOT_SMD:SOT-23" (id 2) (at 144.78 104.14 90)
       (effects (font (size 1.27 1.27)) hide)
     )
@@
     (pin "1")
   )
+  (symbol (lib_id "power:GND") (at 208.28 93.98 0) (unit 1)
+    (in_bom yes) (on_board yes) (fields_autoplaced)
+    (property "Reference" "#PWR?" (id 0) (at 208.28 100.33 0)
+      (effects (font (size 1.27 1.27)) hide)
+    )
+    (property "Value" "GND" (id 1) (at 208.28 98.4234 0))
+    (property "Footprint" "" (id 2) (at 208.28 93.98 0)
+      (effects (font (size 1.27 1.27)) hide)
+    )
+    (property "Datasheet" "" (id 3) (at 208.28 93.98 0)
+      (effects (font (size 1.27 1.27)) hide)
+    )
+    (pin "1")
+  )
   (symbol (lib_id "Device:L") (at 177.8 77.47 90) (unit 1)
     (in_bom yes) (on_board yes) (fields_autoplaced)
     (property "Reference" "L1" (id 0) (at 177.8 73.2622 90))
     (property "Value" "33uH" (id 1) (at 177.8 75.7991 90))
-    (property "Footprint" "Inductor_SMD:L_12x12mm_H4.5mm" (id 2) (at 177.8 77.47 0)
+    (property "Footprint" "Inductor_SMD:L_10.4x10.4_H4.8" (id 2) (at 177.8 77.47 0)
       (effects (font (size 1.27 1.27)) hide)
     )
@@
     (pin "1")
   )
-  (symbol (lib_id "Device:R") (at 194.31 91.44 90) (unit 1)
-    (in_bom yes) (on_board yes) (fields_autoplaced)
-    (property "Reference" "R14" (id 0) (at 194.31 86.7242 90))
-    (property "Value" ".1" (id 1) (at 194.31 89.2611 90))
-    (property "Footprint" "Resistor_SMD:R_1206_3216Metric_Pad1.30x1.75mm_HandSolder" (id 2) (at 194.31 93.218 90)
-      (effects (font (size 1.27 1.27)) hide)
-    )
-    (property "Datasheet" "~" (id 3) (at 194.31 91.44 0)
+  (symbol (lib_id "Device:R") (at 201.93 93.98 90) (unit 1)
+    (in_bom yes) (on_board yes) (fields_autoplaced)
+    (property "Reference" "R?" (id 0) (at 201.93 89.2642 90))
+    (property "Value" ".1" (id 1) (at 201.93 91.8011 90))
+    (property "Footprint" "Resistor_SMD:R_1206_3216Metric_Pad1.30x1.75mm_HandSolder" (id 2) (at 201.93 95.758 90)
+      (effects (font (size 1.27 1.27)) hide)
+    )
+    (property "Datasheet" "~" (id 3) (at 201.93 93.98 0)
       (effects (font (size 1.27 1.27)) hide)
     )
@@
       (effects (font (size 1.27 1.27)) (justify left))
     )
-    (property "Value" "100k" (id 1) (at 137.668 117.2722 0)
+    (property "Value" "47k" (id 1) (at 137.668 117.2722 0)
       (effects (font (size 1.27 1.27)) (justify left))
     )
@@
       (effects (font (size 1.27 1.27)) (justify left))
     )
-    (property "Value" "18k" (id 1) (at 137.668 128.7022 0)
+    (property "Value" "12k" (id 1) (at 137.668 128.7022 0)
       (effects (font (size 1.27 1.27)) (justify left))
     )
@@
       (reference "#PWR0103") (unit 1) (value "VBUS") (footprint "")
     )
-    (path "/15bd5601-cbfa-404a-b2e3-549e2f633b8d"
-      (reference "#PWR0104") (unit 1) (value "GND") (footprint "")
-    )
     (path "/6ebdc5ee-a75a-4d6d-8691-eb4f690c7015"
       (reference "#PWR0105") (unit 1) (value "VBUS") (footprint "")
@@
       (reference "#PWR0131") (unit 1) (value "GND") (footprint "")
     )
+    (path "/7d9d3162-e5d2-4b99-b060-3cd13b2a17e7"
+      (reference "#PWR?") (unit 1) (value "GND") (footprint "")
+    )
     (path "/59f70524-3133-43a1-a30e-50e9f22cf474"
       (reference "BT1") (unit 1) (value "Battery_Cell") (footprint "Connector_PinHeader_2.54mm:PinHeader_1x02_P2.54mm_Vertical")
@@
     )
     (path "/1bf92ec3-2efb-4d05-912b-c9a7f03eabab"
-      (reference "D3") (unit 1) (value "SS34") (footprint "Diode_SMD:D_SMC_Handsoldering")
+      (reference "D3") (unit 1) (value "SS34") (footprint "Diode_SMD:D_SMA_Handsoldering")
     )
     (path "/e54fd964-b82d-40d6-a4d6-64452ac40fc9"
@@
     )
     (path "/860590c4-d7be-44b8-afa6-1e68c7b7f7f1"
-      (reference "L1") (unit 1) (value "33uH") (footprint "Inductor_SMD:L_12x12mm_H4.5mm")
+      (reference "L1") (unit 1) (value "33uH") (footprint "Inductor_SMD:L_10.4x10.4_H4.8")
     )
     (path "/e94c8205-0c46-4260-9314-693da42f22f6"
@@
     )
     (path "/b68b5cb7-e964-4f38-852f-96d6c8b791a5"
-      (reference "R9") (unit 1) (value "100k") (footprint "Resistor_SMD:R_0805_2012Metric_Pad1.20x1.40mm_HandSolder")
+      (reference "R9") (unit 1) (value "47k") (footprint "Resistor_SMD:R_0805_2012Metric_Pad1.20x1.40mm_HandSolder")
     )
     (path "/b799c262-90fc-454e-88e0-ecc81cd25d8b"
-      (reference "R10") (unit 1) (value "18k") (footprint "Resistor_SMD:R_0805_2012Metric_Pad1.20x1.40mm_HandSolder")
+      (reference "R10") (unit 1) (value "12k") (footprint "Resistor_SMD:R_0805_2012Metric_Pad1.20x1.40mm_HandSolder")
     )
     (path "/872ac5d8-2fc1-4581-9696-88f3e00edf63"
       (reference "R11") (unit 1) (value "500") (footprint "Resistor_SMD:R_0805_2012Metric_Pad1.20x1.40mm_HandSolder")
     )
-    (path "/9c958879-1274-4879-9858-bbc083fe6500"
-      (reference "R14") (unit 1) (value ".1") (footprint "Resistor_SMD:R_1206_3216Metric_Pad1.30x1.75mm_HandSolder")
-    )
     (path "/10da1b75-05d9-4012-b6a0-466befa8f37a"
       (reference "R15") (unit 1) (value "1k") (footprint "Resistor_SMD:R_0805_2012Metric_Pad1.20x1.40mm_HandSolder")
@@
       (reference "R23") (unit 1) (value "68k") (footprint "Resistor_SMD:R_0805_2012Metric_Pad1.20x1.40mm_HandSolder")
     )
+    (path "/9747aaa2-ca2b-4739-985d-9003779feb81"
+      (reference "R?") (unit 1) (value ".1") (footprint "Resistor_SMD:R_1206_3216Metric_Pad1.30x1.75mm_HandSolder")
+    )
     (path "/f4611b4c-2e63-4be3-8f43-4356497ca9ae"
       (reference "U1") (unit 1) (value "BSD316") (footprint "Package_TO_SOT_SMD:SOT-363_SC-70-6_Handsoldering")
@@
     )
     (path "/1c720635-3351-4531-a7a0-a3638383571a"
-      (reference "U9") (unit 1) (value "AS431") (footprint "Package_TO_SOT_SMD:SOT-23-5_HandSoldering")
+      (reference "U9") (unit 1) (value "AS431") (footprint "Package_TO_SOT_SMD:SOT-23")
     )
     (path "/0639c911-a4f4-4a91-952f-b8f53266197c"
