File: EDA/Final EDA/driver.kicad_sch (KiCad schematic)
At the start: 8 parts, among them J1 Peltier Connection, U18 slg55021, U2 NL17SZ14, U3 DMT3020LSDQ, U4 DMT3020LSDQ, U6 slg55021, U7 NL17SZ14, U8 NL17SZ14

Commit message: e
Parts:
- removed U7, U8: NL17SZ14, Package_TO_SOT_SMD:SOT-553, symbol 1KicadLib:NL17SZ14
Connections:
- net DRIVER_DIR: now also U4.4 (G)
- net ~DRIVER_DIR_PD: now reaches U18.2 (ON)
- net ~DRIVER_DIR_PD: now also U2.4 (Y), U3.4 (G)
Other:
- moved on the sheet: U2
