File: EDA/Final EDA/HI.kicad_sch (KiCad schematic)
At the start: 4 parts, among them J2 USB_C_Receptacle_USB2.0, SW1 Power Switch

Commit message: e
Connections:
- net VCC_UNREGULATED renamed PWR_SW_N
Changed lines of the file:
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@@
     (stroke (width 0) (type default) (color 0 0 0 0))
   )
-  (wire (pts (xy 101.6 107.95) (xy 125.73 107.95))
+  (wire (pts (xy 101.6 107.95) (xy 129.54 107.95))
     (stroke (width 0) (type default) (color 0 0 0 0))
   )
@@
     (stroke (width 0) (type default) (color 0 0 0 0))
   )
-  (wire (pts (xy 129.54 100.33) (xy 129.54 133.35))
+  (wire (pts (xy 129.54 124.46) (xy 129.54 133.35))
     (stroke (width 0) (type default) (color 0 0 0 0))
   )
@@
     (stroke (width 0) (type default) (color 0 0 0 0))
   )
-  (wire (pts (xy 125.73 95.25) (xy 168.91 95.25))
+  (wire (pts (xy 129.54 115.57) (xy 168.91 115.57))
     (stroke (width 0) (type default) (color 0 0 0 0))
   )
@@
     (stroke (width 0) (type default) (color 0 0 0 0))
   )
-  (wire (pts (xy 125.73 107.95) (xy 125.73 95.25))
+  (wire (pts (xy 129.54 107.95) (xy 129.54 115.57))
     (stroke (width 0) (type default) (color 0 0 0 0))
   )
@@
     (stroke (width 0) (type default) (color 0 0 0 0))
   )
-  (wire (pts (xy 168.91 100.33) (xy 129.54 100.33))
+  (wire (pts (xy 168.91 124.46) (xy 129.54 124.46))
     (stroke (width 0) (type default) (color 0 0 0 0))
   )
-  (hierarchical_label "VCC_UNREGULATED" (shape input) (at 168.91 100.33 0)
-    (effects (font (size 1.27 1.27)) (justify left))
-  )
-  (hierarchical_label "PWR_SW_P" (shape input) (at 168.91 95.25 0)
+  (hierarchical_label "PWR_SW_P" (shape input) (at 168.91 115.57 0)
     (effects (font (size 1.27 1.27)) (justify left))
   )
@@
     (effects (font (size 1.27 1.27)) (justify left))
   )
+  (hierarchical_label "PWR_SW_N" (shape input) (at 168.91 124.46 0)
+    (effects (font (size 1.27 1.27)) (justify left))
+  )

Commit message: E
Parts:
- SW1: footprint Connector_PinHeader_2.54mm:PinHeader_1x02_P2.54mm_Vertical -> Connector_PinHeader_1.27mm:PinHeader_1x02_P1.27mm_Vertical
Changed lines of the file:
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@@
     (property "Reference" "SW1" (id 0) (at 93.98 120.65 90))
     (property "Value" "Power Switch" (id 1) (at 91.44 124.46 90))
-    (property "Footprint" "Connector_PinHeader_2.54mm:PinHeader_1x02_P2.54mm_Vertical" (id 2) (at 101.6 121.92 0)
+    (property "Footprint" "Connector_PinHeader_1.27mm:PinHeader_1x02_P1.27mm_Vertical" (id 2) (at 101.6 121.92 0)
       (effects (font (size 1.27 1.27)) hide)
     )
