File: EDA/Final EDA/InsulinCoolerBoard.kicad_pcb (KiCad board)
At the start: 2 copper layers, 99.1 x 99.1 mm, 87 parts, among them J1 Peltier Connection, J11 PROG_PORT, J2 USB_C_Receptacle_USB2.0, J4 PROG_PORT, J9 PROG_PORT, SW1 Power Switch, U1 ESP32-D-WD-V3, U10 BSD316, U11 BSD316, U12 PC817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

Commit message: e
Parts:
- C17: moved to F.Cu
- moved C17 4.00 mm to (129.4, 75.8), turned to 0 degrees
Routing:
- net /MCU/CELL_DSCHG_3_MCU: track 14.8 -> 35.8 mm
- net PWR_UNREG: track 42.1 -> 56.5 mm
- net /MCU/CELL_DSCHG_2_MCU: track 12.4 -> 25.4 mm
- net +5V: track 34.1 -> 30.1 mm
- net /MCU/DRIVER_EN_MCU: track 41.0 -> 38.0 mm
- net GND: track 9.11 -> 8.32 mm
- net +3V3: track 95.1 -> 95.6 mm, vias 6 -> 7

Commit message: E
Parts:
- removed C15: 10uF, Capacitor_SMD:C_0805_2012Metric_Pad1.18x1.45mm_HandSolder
- C1, C2: footprint Capacitor_SMD:C_0805_2012Metric_Pad1.18x1.45mm_HandSolder -> Capacitor_SMD:C_0603_1608Metric_Pad1.08x0.95mm_HandSolder
- L1: footprint Inductor_SMD:L_0805_2012Metric_Pad1.15x1.40mm_HandSolder -> Inductor_SMD:L_0603_1608Metric_Pad1.05x0.95mm_HandSolder
- R12, R15, R16, R26, R29, R33, R39, R4, R5, U15: moved to B.Cu
- R23: moved to F.Cu
- U12, U13, U14: footprint Package_DIP:DIP-4_W7.62mm -> Package_DIP:DIP-4_W8.89mm_SMDSocket_LongPads; moved to F.Cu
- moved C10 28.2 mm to (156.6, 90.6)
- moved C11 28.2 mm to (165.2, 78.2)
- moved C13 28.2 mm to (174.3, 78.5)
- moved C14 28.2 mm to (175.0, 81.9)
- moved C16 28.2 mm to (162.1, 98.9)
- moved C17 28.2 mm to (157.5, 78.0)
- moved C3 28.2 mm to (153.2, 97.3)
- moved C4 28.2 mm to (153.2, 99.3)
- moved C6 28.2 mm to (152.8, 92.4)
- moved J11 28.2 mm to (168.2, 89.0)
- moved J4 28.2 mm to (166.1, 99.0)
- moved J9 28.2 mm to (153.7, 87.6)
- moved L2 28.2 mm to (169.0, 83.7)
- moved R10 28.2 mm to (159.8, 98.1)
- moved U16 28.2 mm to (169.8, 77.7)
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Routing:
- net /Power Management/BATT: track 94.8 -> 55.7 mm
- net VBUS: track 69.0 -> 33.1 mm, vias 2 -> 3
- net Net-(BT3-Pad2): track 9.28 -> 34.2 mm, vias 1 -> 2
- net /MCU/CELL_DSCHG_3_MCU: track 35.8 -> 13.9 mm
- net Net-(R34-Pad2): track 36.2 -> 16.8 mm, vias 1 -> 3
- net Net-(BT1-Pad2): track 37.7 -> 24.2 mm
- net /MCU/CELL_DSCHG_2_MCU: track 25.4 -> 13.6 mm
- net Net-(BT2-Pad2): track 27.3 -> 17.2 mm
- net Net-(U12-Pad3): track 5.37 -> 12.1 mm, vias 0 -> 1
- net Net-(U11-Pad3): track 5.30 -> 11.5 mm, vias 0 -> 1
- net Net-(U10-Pad3): track 5.20 -> 11.2 mm, vias 0 -> 1
- net Net-(R33-Pad2): track 6.90 -> 12.3 mm, vias 0 -> 2
- net Net-(J2-PadA5): track 0.00 -> 4.65 mm
- net Net-(AE1-Pad1): track 3.92 -> 0.00 mm
- net Net-(R39-Pad2): track 5.74 -> 1.97 mm
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
Commit message: z
Parts:
- moved U2 16.8 mm to (158.0, 69.5), turned to -90 degrees
- moved U8 14.6 mm to (170.2, 70.2), turned to 90 degrees
- moved U7 13.7 mm to (168.4, 71.7), turned to 90 degrees
- moved U18 10.4 mm to (167.5, 68.8), turned to 90 degrees
- moved U6 9.70 mm to (160.7, 66.8), turned to 0 degrees
- moved U4 9.46 mm to (167.5, 66.0), turned to 180 degrees
- moved U3 9.32 mm to (160.9, 67.0), turned to 90 degrees
- moved C9 8.73 mm to (142.4, 70.6)
- moved U19 8.73 mm to (143.2, 65.9)
- moved C12 8.73 mm to (145.8, 70.9)
- moved J1 7.90 mm to (164.7, 61.4), turned to -90 degrees
Routing:
- net PWR_UNREG: track 56.5 -> 16.5 mm
- net /MCU/DRIVER_DIR_MCU: track 45.3 -> 29.5 mm, vias 1 -> 3
- net +5V: track 30.1 -> 19.3 mm
- net /MCU/DRIVER_EN_MCU: track 38.0 -> 28.8 mm
- net Net-(U2-Pad4): track 6.32 -> 4.80 mm
- net Net-(U4-Pad4): track 7.62 -> 6.19 mm
- net Net-(J1-Pad2): track 13.6 -> 14.2 mm
- net GND: track 8.32 -> 7.82 mm, vias 9 -> 8

Commit message: e
Parts:
- removed U7, U8: NL17SZ14, Package_TO_SOT_SMD:SOT-553
- added R2: 10k, Resistor_SMD:R_0805_2012Metric_Pad1.20x1.40mm_HandSolder, B.Cu at (138.9, 95.3)
- C11, C12, C13, C14, C8, C9, U16: moved to B.Cu
- moved R20 64.9 mm to (158.3, 100.2)
- moved R24 64.9 mm to (181.6, 100.2)
- moved TH2 64.9 mm to (167.5, 104.9)
- moved TH3 64.9 mm to (181.6, 104.6)
- moved R21 64.9 mm to (167.5, 99.8)
- moved TH1 64.9 mm to (158.2, 104.8)
- moved SW1 50.2 mm to (140.8, 92.4)
- moved C14 38.5 mm to (136.6, 80.6), turned to 90 degrees
- moved C13 38.3 mm to (136.6, 84.5), turned to -90 degrees
- moved C8 33.0 mm to (132.4, 92.1), turned to 180 degrees
- moved U16 30.5 mm to (139.6, 82.6), turned to 0 degrees
- moved L2 30.1 mm to (138.8, 83.8), turned to 180 degrees
- moved C16 30.0 mm to (132.1, 98.3)
- moved R10 30.0 mm to (129.8, 97.6)
- moved C10 30.0 mm to (126.7, 90.0)
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Connections:
- BT1 pad 1: /Power Management/BATT -> PWR_UNREG
- C21 pad 1: /Power Management/BATT -> PWR_UNREG
- D4 pad 1: /Power Management/BATT -> PWR_UNREG
- R12 pad 1: /Power Management/BATT -> PWR_UNREG
- R22 pad 1: /Power Management/BATT -> PWR_UNREG
- R30 pad 1: /Power Management/BATT -> PWR_UNREG
- SW1 pad 1: PWR_UNREG -> +3V3
- SW1 pad 2: /Power Management/BATT -> /MCU/PWR_SW_P_MCU
- U1 pad 17: unconnected-(U1-Pad17) -> /MCU/PWR_SW_P_MCU
- U12 pad 4: /Power Management/BATT -> PWR_UNREG
- U18 pad 2: Net-(U18-Pad2) -> /Peltier Driver/~DRIVER_DIR_PD
- U2 pad 4: Net-(U2-Pad4) -> /Peltier Driver/~DRIVER_DIR_PD
- U3 pad 4: Net-(U2-Pad4) -> /Peltier Driver/~DRIVER_DIR_PD
- U4 pad 4: Net-(U4-Pad4) -> /MCU/DRIVER_DIR_MCU
Routing:
- net /Power Management/BATT: track 55.7 -> 0.00 mm, vias 1 -> 0
- net PWR_UNREG: track 16.5 -> 70.8 mm, vias 2 -> 5
- net /MCU/CELL_DSCHG_3_MCU: track 13.9 -> 47.0 mm, vias 1 -> 3
- net /MCU/CELL_DSCHG_2_MCU: track 13.6 -> 31.9 mm, vias 1 -> 3
- net +5V: track 19.3 -> 3.99 mm, vias 2 -> 1
- net Net-(C11-Pad1): track 12.8 -> 0.00 mm, vias 0 -> 2
- net /MCU/CELL_MEAS_3_MCU: track 28.3 -> 17.6 mm
- net /MCU/PWR_SW_P_MCU: track 0.00 -> 10.6 mm
- net /MCU/CELL_MEAS_2_MCU: track 26.3 -> 16.1 mm
- net /MCU/DRIVER_EN_MCU: track 28.8 -> 20.1 mm
- net /Peltier Driver/~DRIVER_DIR_PD: track 0.00 -> 8.24 mm, vias 0 -> 1
- net /MCU/IO0: track 4.97 -> 13.2 mm
- net Net-(U4-Pad4): track 6.19 -> 0.00 mm
- net /MCU/CELL_MEAS_1_MCU: track 20.2 -> 14.7 mm
- net Net-(U2-Pad4): track 4.80 -> 0.00 mm, vias 1 -> 0
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
Commit message: E
Parts:
- J11, J4, J9, SW1: footprint Connector_PinHeader_2.54mm:PinHeader_1x02_P2.54mm_Vertical -> Connector_PinHeader_1.27mm:PinHeader_1x02_P1.27mm_Vertical
- R18, R19: moved to F.Cu
- R20, R21, R24: moved to B.Cu
- TH1, TH2, TH3: footprint Resistor_SMD:R_0805_2012Metric_Pad1.20x1.40mm_HandSolder -> Connector_PinHeader_1.27mm:PinHeader_1x02_P1.27mm_Vertical
- moved R24 43.7 mm to (138.1, 96.2)
- moved TH3 42.7 mm to (140.1, 94.7), turned to 90 degrees
- moved TH2 30.5 mm to (140.1, 91.5), turned to 90 degrees
- moved R21 30.2 mm to (138.3, 92.3)
- moved TH1 24.5 mm to (140.2, 88.2), turned to 90 degrees
- moved R20 23.2 mm to (138.3, 88.5)
- moved C1 17.6 mm to (125.8, 102.0), turned to 180 degrees
- moved C2 16.8 mm to (125.8, 97.0), turned to 180 degrees
- moved AE1 16.5 mm to (126.6, 107.1)
- moved L1 14.5 mm to (126.7, 99.5)
- moved R18 8.47 mm to (115.0, 78.3), turned to 0 degrees
- moved R19 7.96 mm to (119.1, 82.1), turned to -90 degrees
- moved R17 6.65 mm to (99.6, 81.1), turned to 0 degrees
- moved SW1 5.43 mm to (135.5, 91.4), turned to 90 degrees
- moved R26 3.75 mm to (116.7, 74.7), turned to 0 degrees
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Connections:
- U1 pad 20: /MCU/CELL_MEAS_3_MCU -> /MCU/CELL_MEAS_1_MCU
- U1 pad 22: /MCU/CELL_MEAS_1_MCU -> /MCU/CELL_MEAS_3_MCU
Routing:
- net PWR_UNREG: track 70.8 -> 123.2 mm
- net /MCU/CELL_MEAS_3_MCU: track 17.6 -> 42.6 mm, vias 1 -> 2
- net Net-(R39-Pad2): track 1.97 -> 25.5 mm
- net +5V: track 3.99 -> 22.6 mm, vias 1 -> 2
- net /MCU/DRIVER_EN_MCU: track 20.1 -> 35.3 mm
- net /MCU/CELL_MEAS_2_MCU: track 16.1 -> 31.2 mm, vias 0 -> 1
- net /MCU/CELL_MEAS_1_MCU: track 14.7 -> 29.8 mm
- net +3V3: track 91.8 -> 78.7 mm, vias 8 -> 7
- net /MCU/DRIVER_DIR_MCU: track 29.3 -> 39.6 mm
- net /MCU/CELL_DSCHG_2_MCU: track 31.9 -> 22.1 mm, vias 3 -> 2
- net /MCU/CELL_DSCHG_3_MCU: track 47.0 -> 37.3 mm, vias 3 -> 1
- net /MCU/TEMP_SENSE_1: track 6.13 -> 15.3 mm
- net /MCU/TEMP_SENSE_2: track 6.99 -> 13.2 mm
- net Net-(AE1-Pad1): track 0.00 -> 5.28 mm
- net Net-(R18-Pad1): track 4.81 -> 9.88 mm, vias 1 -> 0
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Other:
- board size 99.1 x 99.1 mm -> 46.3 x 45.3 mm
- board text added: "Insulin Cooler"
- board text added: "Joesphan Lu"
- board text removed: "3V3"
- board text removed: "5V"
- board text removed: "DIRT"
- board text removed: "PWR_UNREG"
- board text removed: "VBUS"
