File: EDA/Final EDA/pwrmngmt.kicad_sch (KiCad schematic)
At the start: 45 parts, among them U10 BSD316, U11 BSD316, U12 PC817, U13 PC817, U14 PC817, U15 AS431, U16 AP63203WU, U17 XL6009, U19 HT75xx-1-SOT89, U5 LM324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

Commit message: E
Parts:
- removed C15: 10uF, Capacitor_SMD:C_0805_2012Metric_Pad1.18x1.45mm_HandSolder, symbol Device:C
- U12, U13, U14: footprint Package_DIP:DIP-4_W7.62mm -> Package_DIP:DIP-4_W8.89mm_SMDSocket_LongPads
Changed lines of the file:
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@@
     (comment 1 "Engineer/Draftsman: Joesphan Lu")
   )
-  (junction (at 116.84 140.97) (diameter 0) (color 0 0 0 0)
-  )
   (junction (at 48.26 80.01) (diameter 0) (color 0 0 0 0)
   )
@@
   (junction (at 226.06 96.52) (diameter 0) (color 0 0 0 0)
   )
-  (junction (at 116.84 158.75) (diameter 0) (color 0 0 0 0)
-  )
   (junction (at 21.59 154.94) (diameter 0) (color 0 0 0 0)
   )
@@
     (stroke (width 0) (type default) (color 0 0 0 0))
   )
-  (wire (pts (xy 130.81 156.21) (xy 130.81 158.75))
-    (stroke (width 0) (type default) (color 0 0 0 0))
-  )
   (polyline (pts (xy 281.94 13.97) (xy 281.94 67.31))
     (stroke (width 0) (type default) (color 0 0 0 0))
@@
     (stroke (width 0) (type default) (color 0 0 0 0))
   )
-  (wire (pts (xy 116.84 158.75) (xy 116.84 161.29))
-    (stroke (width 0) (type default) (color 0 0 0 0))
-  )
   (wire (pts (xy 125.73 82.55) (xy 121.92 82.55))
     (stroke (width 0) (type default) (color 0 0 0 0))
@@
     (stroke (width 0) (type default) (color 0 0 0 0))
   )
-  (wire (pts (xy 116.84 140.97) (xy 130.81 140.97))
+  (wire (pts (xy 109.22 140.97) (xy 130.81 140.97))
     (stroke (width 0) (type default) (color 0 0 0 0))
   )
@@
     (stroke (width 0) (type default) (color 0 0 0 0))
   )
-  (wire (pts (xy 116.84 148.59) (xy 116.84 140.97))
-    (stroke (width 0) (type default) (color 0 0 0 0))
-  )
   (wire (pts (xy 21.59 142.24) (xy 21.59 144.78))
     (stroke (width 0) (type default) (color 0 0 0 0))
@@
     (stroke (width 0) (type default) (color 0 0 0 0))
   )
-  (wire (pts (xy 116.84 158.75) (xy 130.81 158.75))
+  (wire (pts (xy 130.81 156.21) (xy 130.81 162.56))
     (stroke (width 0) (type default) (color 0 0 0 0))
   )
@@
     (stroke (width 0) (type default) (color 0 0 0 0))
   )
-  (wire (pts (xy 109.22 140.97) (xy 116.84 140.97))
-    (stroke (width 0) (type default) (color 0 0 0 0))
-  )
   (wire (pts (xy 90.17 149.86) (xy 90.17 140.97))
     (stroke (width 0) (type default) (color 0 0 0 0))
   )
   (wire (pts (xy 160.02 40.64) (xy 156.21 40.64))
-    (stroke (width 0) (type default) (color 0 0 0 0))
-  )
-  (wire (pts (xy 116.84 156.21) (xy 116.84 158.75))
     (stroke (width 0) (type default) (color 0 0 0 0))
   )
@@
     (pin "3")
   )
-  (symbol (lib_id "Device:C") (at 116.84 152.4 0) (mirror y) (unit 1)
-    (in_bom yes) (on_board yes)
-    (property "Reference" "C15" (id 0) (at 113.919 151.2316 0)
-      (effects (font (size 1.27 1.27)) (justify left))
-    )
-    (property "Value" "10uF" (id 1) (at 124.46 152.4 0)
-      (effects (font (size 1.27 1.27)) (justify left))
-    )
-    (property "Footprint" "Capacitor_SMD:C_0805_2012Metric_Pad1.18x1.45mm_HandSolder" (id 2) (at 115.8748 156.21 0)
-      (effects (font (size 1.27 1.27)) hide)
-    )
-    (property "Datasheet" "~" (id 3) (at 116.84 152.4 0)
-      (effects (font (size 1.27 1.27)) hide)
-    )
-    (pin "1")
-    (pin "2")
-  )
   (symbol (lib_id "1KicadLib:XL6009") (at 77.47 156.21 0) (unit 1)
     (in_bom yes) (on_board yes) (fields_autoplaced)
@@
     (property "Reference" "U13" (id 0) (at 58.42 56.515 0))
     (property "Value" "PC817" (id 1) (at 58.42 58.8264 0))
-    (property "Footprint" "Package_DIP:DIP-4_W7.62mm" (id 2) (at 63.5 69.85 0)
+    (property "Footprint" "Package_DIP:DIP-4_W8.89mm_SMDSocket_LongPads" (id 2) (at 63.5 69.85 0)
       (effects (font (size 1.27 1.27) italic) (justify left) hide)
     )
@@
     (pin "2")
   )
-  (symbol (lib_id "power:GND") (at 116.84 161.29 0) (unit 1)
-    (in_bom yes) (on_board yes) (fields_autoplaced)
-    (property "Reference" "#PWR0156" (id 0) (at 116.84 167.64 0)
-      (effects (font (size 1.27 1.27)) hide)
-    )
-    (property "Value" "GND" (id 1) (at 116.84 165.7334 0))
-    (property "Footprint" "" (id 2) (at 116.84 161.29 0)
-      (effects (font (size 1.27 1.27)) hide)
-    )
-    (property "Datasheet" "" (id 3) (at 116.84 161.29 0)
+  (symbol (lib_id "power:GND") (at 130.81 162.56 0) (unit 1)
+    (in_bom yes) (on_board yes) (fields_autoplaced)
+    (property "Reference" "#PWR0156" (id 0) (at 130.81 168.91 0)
+      (effects (font (size 1.27 1.27)) hide)
+    )
+    (property "Value" "GND" (id 1) (at 130.81 167.0034 0))
+    (property "Footprint" "" (id 2) (at 130.81 162.56 0)
+      (effects (font (size 1.27 1.27)) hide)
+    )
+    (property "Datasheet" "" (id 3) (at 130.81 162.56 0)
       (effects (font (size 1.27 1.27)) hide)
     )
@@
     (property "Reference" "U14" (id 0) (at 58.42 84.455 0))
     (property "Value" "PC817" (id 1) (at 58.42 86.7664 0))
-    (property "Footprint" "Package_DIP:DIP-4_W7.62mm" (id 2) (at 63.5 97.79 0)
+    (property "Footprint" "Package_DIP:DIP-4_W8.89mm_SMDSocket_LongPads" (id 2) (at 63.5 97.79 0)
       (effects (font (size 1.27 1.27) italic) (justify left) hide)
     )
@@
     (property "Reference" "U12" (id 0) (at 58.42 27.305 0))
     (property "Value" "PC817" (id 1) (at 58.42 29.6164 0))
-    (property "Footprint" "Package_DIP:DIP-4_W7.62mm" (id 2) (at 63.5 40.64 0)
+    (property "Footprint" "Package_DIP:DIP-4_W8.89mm_SMDSocket_LongPads" (id 2) (at 63.5 40.64 0)
       (effects (font (size 1.27 1.27) italic) (justify left) hide)
     )

Commit message: e
Connections:
- net VCC_UNREGULATED is gone; now on net PWR_UNREG: C9.1, U16.2 (EN), U16.3 (IN), U19.2 (VIN)
- net PWR_SW_P renamed PWR_UNREG
Changed lines of the file:
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@@
-    (stroke (width 0) (type default) (color 0 0 0 0))
-  )
-  (wire (pts (xy 156.21 25.4) (xy 161.29 25.4))
     (stroke (width 0) (type default) (color 0 0 0 0))
   )
@@
     (stroke (width 0) (type default) (color 0 0 0 0))
   )
+  (wire (pts (xy 156.21 34.29) (xy 161.29 34.29))
+    (stroke (width 0) (type default) (color 0 0 0 0))
+  )
   (wire (pts (xy 243.84 96.52) (xy 226.06 96.52))
     (stroke (width 0) (type default) (color 0 0 0 0))
@@
   )
   (wire (pts (xy 27.94 173.99) (xy 34.29 173.99))
-    (stroke (width 0) (type default) (color 0 0 0 0))
-  )
-  (wire (pts (xy 156.21 31.75) (xy 158.75 31.75))
     (stroke (width 0) (type default) (color 0 0 0 0))
   )
@@
     (effects (font (size 3 3)) (justify left bottom))
   )
-  (label "PWR__UNREG_PWRMG" (at 158.75 31.75 0)
-    (effects (font (size 1.27 1.27)) (justify left bottom))
-  )
   (label "BATT" (at 21.59 20.32 0)
     (effects (font (size 1.27 1.27)) (justify left bottom))
   )
-  (label "PWR__UNREG_PWRMG" (at 185.42 24.13 0)
-    (effects (font (size 1.27 1.27)) (justify left bottom))
-  )
   (label "BATT" (at 21.59 142.24 0)
     (effects (font (size 1.27 1.27)) (justify left bottom))
@@
     (effects (font (size 1.27 1.27)) (justify left bottom))
   )
-  (label "PWR__UNREG_PWRMG" (at 204.47 74.93 0)
+  (label "BATT" (at 185.42 24.13 0)
     (effects (font (size 1.27 1.27)) (justify left bottom))
   )
@@
     (effects (font (size 1.27 1.27)) (justify left bottom))
   )
-  (label "BATT" (at 161.29 25.4 0)
+  (label "BATT" (at 204.47 74.93 0)
     (effects (font (size 1.27 1.27)) (justify left bottom))
   )
@@
     (effects (font (size 1.27 1.27)) (justify left bottom))
   )
+  (label "BATT" (at 161.29 34.29 0)
+    (effects (font (size 1.27 1.27)) (justify left bottom))
+  )
   (label "3V3" (at 160.02 40.64 0)
     (effects (font (size 1.27 1.27)) (justify left bottom))
-  )
-  (hierarchical_label "PWR_SW_P" (shape input) (at 156.21 25.4 180)
-    (effects (font (size 1.27 1.27)) (justify right))
-  )
-  (hierarchical_label "VCC_UNREGULATED" (shape input) (at 156.21 31.75 180)
-    (effects (font (size 1.27 1.27)) (justify right))
   )
   (hierarchical_label "5V" (shape input) (at 156.21 45.72 180)
@@
     (effects (font (size 1.27 1.27)) (justify right))
   )
+  (hierarchical_label "PWR_UNREG" (shape input) (at 156.21 34.29 180)
+    (effects (font (size 1.27 1.27)) (justify right))
+  )

Commit message: code done ish
Parts:
- R34, R7: value 12.5k -> 30k
- R5, R6: value 1k -> 2.4k
Changed lines of the file:
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@@
     (in_bom yes) (on_board yes) (fields_autoplaced)
     (property "Reference" "R6" (id 0) (at 49.53 114.6642 90))
-    (property "Value" "1k" (id 1) (at 49.53 117.2011 90))
+    (property "Value" "2.4k" (id 1) (at 49.53 117.2011 90))
     (property "Footprint" "Resistor_SMD:R_0805_2012Metric_Pad1.20x1.40mm_HandSolder" (id 2) (at 49.53 117.602 90)
       (effects (font (size 1.27 1.27)) hide)
@@
       (effects (font (size 1.27 1.27)) (justify left))
     )
-    (property "Value" "1k" (id 1) (at 44.0178 126.238 0)
+    (property "Value" "2.4k" (id 1) (at 44.0178 126.238 0)
       (effects (font (size 1.27 1.27)) (justify left))
     )
@@
     (in_bom yes) (on_board yes) (fields_autoplaced)
     (property "Reference" "R34" (id 0) (at 62.23 105.7742 90))
-    (property "Value" "12.5k" (id 1) (at 62.23 108.3111 90))
+    (property "Value" "30k" (id 1) (at 62.23 108.3111 90))
     (property "Footprint" "Resistor_SMD:R_0805_2012Metric_Pad1.20x1.40mm_HandSolder" (id 2) (at 62.23 112.268 90)
       (effects (font (size 1.27 1.27)) hide)
@@
       (effects (font (size 1.27 1.27)) (justify left))
     )
-    (property "Value" "12.5k" (id 1) (at 53.848 133.7822 0)
-      (effects (font (size 1.27 1.27)) (justify left))
-    )
+    (property "Value" "30k" (id 1) (at 53.848 133.7822 0)
+      (effects (font (size 1.27 1.27)) (justify left))
+    )
