File: EDA/Final EDA/tempsensor.kicad_sch (KiCad schematic)
At the start: 6 parts

Commit message: E
Parts:
- TH1, TH2, TH3: footprint Resistor_SMD:R_0805_2012Metric_Pad1.20x1.40mm_HandSolder -> Connector_PinHeader_1.27mm:PinHeader_1x02_P1.27mm_Vertical
Other:
- moved on the sheet: R20, R21, R24, TH1, TH2, TH3

Commit message: code done ish
Parts:
- R20, R21, R24: value 90k -> 10k
